File: Hardware/CPU Card/CPU Card.sch (KiCad schematic (older format))
At the start: 9 parts, among them IC1 W65C02S6TPG-14

Commit message: Cleanup
Parts:
- removed C1: 100nF, CPU Card:C025-030X050, symbol CPU_Card-eagle-import:C-US025-030X050
- removed CONN1: 6502CARDEDGE, CPU Card:6502CARDEDGE, symbol CPU_Card-eagle-import:6502CARDEDGE
- removed IC1: W65C02S6TPG-14, CPU Card:DIP1524W56P254L5207H508Q40N, symbol CPU_Card-eagle-import:W65C02S6TPG-14
- removed JP1: PINHD-2X3, CPU Card:2X03, symbol CPU_Card-eagle-import:PINHD-2X3
- removed R1, R2, R3, R4, R5: 1k, CPU Card:RESAD724W46L381D178B, symbol CPU_Card-eagle-import:R-USAXIAL-7.2MM-PITCH
- added C1: 100nF, Capacitor_SMD:C_0805_2012Metric, symbol Device:C
- added CONN1: 6502CARDEDGE, CPU Card:6502CARDEDGE, symbol CPU_Card:6502CARDEDGE
- added IC1: W65C02S6TPG-14, CPU Card:DIP1524W56P254L5207H508Q40N, symbol CPU_Card:W65C02S6TPG-14
- added J1: Conn_02x02_Odd_Even, symbol Connector_Generic:Conn_02x02_Odd_Even
- added R1, R2, R3, R4, R5: 1k, Resistor_SMD:R_0805_2012Metric, symbol Device:R
Connections:
- net labels added: R~W, ~IRQ, ~ML, ~NMI, ~RES
- net labels removed: EXP1, IRQB, MLB, NMIB, PHI2O, RESB, RWB, VPB, _PHI1O
- wire segments 100 -> 99
- no-connect marks 0 -> 3

Commit message: Working on schematic capture
Parts:
- IC1: footprint CPU Card:DIP1524W56P254L5207H508Q40N -> Package_DIP:DIP-40_W15.24mm_Socket_LongPads
- J1: footprint (none) -> Connector_PinHeader_2.54mm:PinHeader_2x02_P2.54mm_Vertical
Changed lines of the file:
@@
 F 0 "IC1" H 5550 3086 59  0000 C CNN
 F 1 "W65C02S6TPG-14" H 5550 2981 59  0000 C CNN
-F 2 "CPU Card:DIP1524W56P254L5207H508Q40N" H 4950 2750 50  0001 C CNN
+F 2 "Package_DIP:DIP-40_W15.24mm_Socket_LongPads" H 4950 2750 50  0001 C CNN
 F 3 "" H 4950 2750 50  0001 C CNN
 	1    4950 2750
@@
 F 0 "J1" H 5550 1925 50  0000 C CNN
 F 1 "Conn_02x02_Odd_Even" H 5550 1926 50  0001 C CNN
-F 2 "" H 5500 1800 50  0001 C CNN
+F 2 "Connector_PinHeader_2.54mm:PinHeader_2x02_P2.54mm_Vertical" H 5500 1800 50  0001 C CNN
 F 3 "~" H 5500 1800 50  0001 C CNN
 	1    5500 1800
@@
 U 1 1 605F5B01
 P 3000 3650
-F 0 "CONN1" H 3000 4730 59  0000 C CNN
-F 1 "6502CARDEDGE" H 3000 3650 50  0001 C CNN
+F 0 "CONN1" H 3000 4800 59  0000 C CNN
+F 1 "6502CARDEDGE" H 3000 4700 50  0000 C CNN
 F 2 "CPU Card:6502CARDEDGE" H 3000 3650 50  0001 C CNN
 F 3 "" H 3000 3650 50  0001 C CNN
@@
 NoConn ~ 3600 2850
 $Comp
-L power:PWR_FLAG #FLG?
+L power:PWR_FLAG #FLG0102
 U 1 1 60707BD0
 P 8400 4600
-F 0 "#FLG?" H 8400 4675 50  0001 C CNN
+F 0 "#FLG0102" H 8400 4675 50  0001 C CNN
 F 1 "PWR_FLAG" V 8400 4727 50  0001 L CNN
 F 2 "" H 8400 4600 50  0001 C CNN

Commit message: Layout CPU card
Parts:
- added JP1, JP2: SolderJumper_2_Open, Jumper:SolderJumper-2_P1.3mm_Open_RoundedPad1.0x1.5mm, symbol Jumper:SolderJumper_2_Open
Connections:
- net EXP0: now also JP2.2 (B)
- net PHI1O: now also JP1.2 (B)
- net at IC1.1 (VPB), J1.3 (Pin_3): now also JP2.1 (A)
- net at IC1.3 (PHI1O), J1.1 (Pin_1): now also JP1.1 (A)
Changed lines of the file:
@@
 	4800 2750 4800 1900
 Wire Wire Line
-	4800 1900 5300 1900
+	4800 1900 5250 1900
 Wire Wire Line
 	4950 2950 4700 2950
@@
 	4700 2950 4700 1800
 Wire Wire Line
-	4700 1800 5300 1800
-Wire Wire Line
-	5800 1800 5950 1800
-Wire Wire Line
-	5800 1900 5950 1900
+	4700 1800 5250 1800
+Wire Wire Line
+	5800 1800 5850 1800
+Wire Wire Line
+	5800 1900 5850 1900
 Text GLabel 5950 1900 2    50   Output ~ 0
 EXP0
@@
 Wire Wire Line
 	8400 4600 8400 4750
+$Comp
+L Jumper:SolderJumper_2_Open JP2
+U 1 1 606F23BA
+P 5550 2150
+F 0 "JP2" H 5550 2263 50  0000 C CNN
+F 1 "SolderJumper_2_Open" H 5550 2264 50  0001 C CNN
+F 2 "Jumper:SolderJumper-2_P1.3mm_Open_RoundedPad1.0x1.5mm" H 5550 2150 50  0001 C CNN
+F 3 "~" H 5550 2150 50  0001 C CNN
+	1    5550 2150
+	1    0    0    -1
+$EndComp
+$Comp
+L Jumper:SolderJumper_2_Open JP1
+U 1 1 606F2C26
+P 5550 1550
+F 0 "JP1" H 5550 1663 50  0000 C CNN
+F 1 "SolderJumper_2_Open" H 5550 1664 50  0001 C CNN
+F 2 "Jumper:SolderJumper-2_P1.3mm_Open_RoundedPad1.0x1.5mm" H 5550 1550 50  0001 C CNN
+F 3 "~" H 5550 1550 50  0001 C CNN
+	1    5550 1550
+	1    0    0    -1
+$EndComp
+Wire Wire Line
+	5700 1550 5850 1550
+Wire Wire Line
+	5850 1550 5850 1800
+Connection ~ 5850 1800
+Wire Wire Line
+	5850 1800 5950 1800
+Wire Wire Line
+	5400 1550 5250 1550
+Wire Wire Line
+	5250 1550 5250 1800
+Connection ~ 5250 1800
+Wire Wire Line
+	5250 1800 5300 1800
+Wire Wire Line
+	5400 2150 5250 2150
+Wire Wire Line
+	5250 2150 5250 1900
+Connection ~ 5250 1900
+Wire Wire Line
+	5250 1900 5300 1900
+Wire Wire Line
+	5700 2150 5850 2150
+Wire Wire Line
+	5850 2150 5850 1900
 Wire Bus Line
 	4200 2650 4200 5300
@@
 Wire Bus Line
 	1800 2650 1800 5300
+Connection ~ 5850 1900
+Wire Wire Line
+	5850 1900 5950 1900
 $EndSCHEMATC

Commit message: Generate production files
Parts:
- C1: LCSC (none) -> C49678
- R1, R2, R3, R4, R5: LCSC (none) -> C17513
Changed lines of the file:
@@
 F 2 "Resistor_SMD:R_0805_2012Metric" V 8730 2850 50  0001 C CNN
 F 3 "~" H 8800 2850 50  0001 C CNN
+F 4 "C17513" H 8800 2850 50  0001 C CNN "LCSC"
 	1    8800 2850
 	0    1    1    0
@@
 F 2 "Resistor_SMD:R_0805_2012Metric" V 8730 3150 50  0001 C CNN
 F 3 "~" H 8800 3150 50  0001 C CNN
+F 4 "C17513" H 8800 3150 50  0001 C CNN "LCSC"
 	1    8800 3150
 	0    1    1    0
@@
 F 2 "Resistor_SMD:R_0805_2012Metric" V 8730 3450 50  0001 C CNN
 F 3 "~" H 8800 3450 50  0001 C CNN
+F 4 "C17513" H 8800 3450 50  0001 C CNN "LCSC"
 	1    8800 3450
 	0    1    1    0
@@
 F 2 "Resistor_SMD:R_0805_2012Metric" V 8730 3750 50  0001 C CNN
 F 3 "~" H 8800 3750 50  0001 C CNN
+F 4 "C17513" H 8800 3750 50  0001 C CNN "LCSC"
 	1    8800 3750
 	0    1    1    0
@@
 F 2 "Resistor_SMD:R_0805_2012Metric" V 8730 4050 50  0001 C CNN
 F 3 "~" H 8800 4050 50  0001 C CNN
+F 4 "C17513" H 8800 4050 50  0001 C CNN "LCSC"
 	1    8800 4050
 	0    1    1    0
@@
 F 2 "Capacitor_SMD:C_0805_2012Metric" H 8438 4200 50  0001 C CNN
 F 3 "~" H 8400 4350 50  0001 C CNN
+F 4 "C49678" H 8400 4350 50  0001 C CNN "LCSC"
 	1    8400 4350
 	1    0    0    -1
@@
 Wire Wire Line
 	5850 2150 5850 1900
+Connection ~ 5850 1900
+Wire Wire Line
+	5850 1900 5950 1900
 Wire Bus Line
 	4200 2650 4200 5300
@@
 Wire Bus Line
 	1800 2650 1800 5300
-Connection ~ 5850 1900
-Wire Wire Line
-	5850 1900 5950 1900
 $EndSCHEMATC

Commit message: CPU Card revisions
Parts:
- added C2: 100nF, Capacitor_SMD:C_0805_2012Metric, symbol Device:C
- added J2: Conn_01x02, Connector_PinHeader_2.54mm:PinHeader_1x02_P2.54mm_Vertical, symbol Connector_Generic:Conn_01x02
- added JP3: SolderJumper_2_Open, Jumper:SolderJumper-2_P1.3mm_Open_RoundedPad1.0x1.5mm, symbol Jumper:SolderJumper_2_Open
- added X1: CXO_DIP14, Oscillator:Oscillator_DIP-14, symbol Oscillator:CXO_DIP14
Connections:
- net GND: now also C2.2, X1.7 (GND)
- net PHI2: now also J2.2 (Pin_2), JP3.2 (B)
- net VCC: now also C2.1, X1.14 (Vcc)
- net at J1.1 (Pin_1), JP1.1 (A): now also IC1.7 (SYNC); no longer IC1.3 (PHI1O)
- net EXP0 renamed EXP3
- net EXP3: now also CONN1.EXP3; no longer CONN1.EXP0
- net PHI1O renamed EXP2
- net EXP2: now also CONN1.EXP2; no longer CONN1.EXP3
- removed net SYNC: CONN1.EXP2, IC1.7 (SYNC)
- new net: J2.1 (Pin_1), JP3.1 (A), X1.8 (OUT)
- no-connect marks 3 -> 6
Changed lines of the file:
@@
 Title "6502 CPU Card"
 Date "2021-03-27"
-Rev "1"
+Rev "1.1"
 Comp "A.C. Wright Design"
 Comment1 ""
@@
 	4800 1900 5250 1900
 Wire Wire Line
-	4950 2950 4700 2950
-Wire Wire Line
-	4700 2950 4700 1800
-Wire Wire Line
 	4700 1800 5250 1800
 Wire Wire Line
@@
 	5800 1900 5850 1900
 Text GLabel 5950 1900 2    50   Output ~ 0
-EXP0
+EXP3
 Text GLabel 5950 1800 2    50   Output ~ 0
-PHI1O
+EXP2
 Wire Bus Line
 	4200 5300 6900 5300
@@
 	6900 2650 6800 2750
 Entry Wire Line
-	6900 2950 6800 3050
-Entry Wire Line
 	6900 3050 6800 3150
 Entry Wire Line
@@
 	4200 3150 4300 3250
 Entry Wire Line
-	4200 3250 4300 3350
-Entry Wire Line
 	4200 3350 4300 3450
 Entry Wire Line
@@
 Entry Wire Line
 	4200 4550 4300 4650
-Entry Wire Line
-	4200 2850 4100 2950
 Entry Wire Line
 	4200 2950 4100 3050
@@
 	6150 2750 6800 2750
 Wire Wire Line
-	6150 3050 6800 3050
-Wire Wire Line
 	6150 3150 6800 3150
 Wire Wire Line
@@
 	4300 3250 4950 3250
 Wire Wire Line
-	4950 3350 4300 3350
-Wire Wire Line
 	4300 3450 4950 3450
 Wire Wire Line
@@
 Wire Wire Line
 	4300 4650 4950 4650
-Wire Wire Line
-	4100 2950 3600 2950
 Wire Wire Line
 	3600 3050 4100 3050
@@
 PHI2
 Text Label 1950 3650 0    50   ~ 0
-PHI1O
+EXP3
 Text Label 1950 3750 0    50   ~ 0
-SYNC
+EXP2
 Text Label 1950 3850 0    50   ~ 0
 D7
@@
 Text Label 1950 4650 0    50   ~ 0
 VCC
-Text Label 4050 2950 2    50   ~ 0
-EXP0
 Text Label 4050 3050 2    50   ~ 0
 A15
@@
 Text Label 6750 2750 2    50   ~ 0
 ~RES
-Text Label 6750 3050 2    50   ~ 0
-PHI2
 Text Label 6750 3150 2    50   ~ 0
 BE
@@
 Text Label 4350 3250 0    50   ~ 0
 ~NMI
-Text Label 4350 3350 0    50   ~ 0
-SYNC
 Text Label 4350 3450 0    50   ~ 0
 VCC
@@
 Wire Wire Line
 	5850 1900 5950 1900
+NoConn ~ 4950 2950
+Entry Wire Line
+	6900 2950 6800 3050
+Text Label 6750 3050 2    50   ~ 0
+PHI2
+Wire Wire Line
+	6150 3050 6800 3050
+Wire Wire Line
+	4700 3350 4950 3350
+Wire Wire Line
+	4700 1800 4700 3350
+$Comp
+L Oscillator:CXO_DIP14 X1
+U 1 1 609BE213
+P 2500 6650
+F 0 "X1" H 2200 6950 50  0000 L CNN
+F 1 "CXO_DIP14" H 2844 6605 50  0001 L CNN
+F 2 "Oscillator:Oscillator_DIP-14" H 2950 6300 50  0001 C CNN
+F 3 "http://cdn-reichelt.de/documents/datenblatt/B400/OSZI.pdf" H 2400 6650 50  0001 C CNN
+	1    2500 6650
+	1    0    0    -1
+$EndComp
+NoConn ~ 2200 6650
+Text GLabel 2500 6100 1    50   Input ~ 0
+VCC
+Wire Wire Line
+	2500 6350 2500 6200
+Wire Wire Line
+	2500 6950 2500 7100
+$Comp
+L power:GND #PWR01
+U 1 1 609D8514
+P 2500 7200
+F 0 "#PWR01" H 2500 6950 50  0001 C CNN
+F 1 "GND" H 2505 7027 50  0000 C CNN
+F 2 "" H 2500 7200 50  0001 C CNN
+F 3 "" H 2500 7200 50  0001 C CNN
+	1    2500 7200
+	1    0    0    -1
+$EndComp
+Text GLabel 3550 6650 2    50   Output ~ 0
+PHI2
+$Comp
+L Connector_Generic:Conn_01x02 J2
+U 1 1 609FEB8E
+P 3100 6350
+F 0 "J2" V 3100 6550 50  0000 R CNN
+F 1 "Conn_01x02" V 2973 6162 50  0001 R CNN
+F 2 "Connector_PinHeader_2.54mm:PinHeader_1x02_P2.54mm_Vertical" H 3100 6350 50  0001 C CNN
+F 3 "~" H 3100 6350 50  0001 C CNN
+	1    3100 6350
+	0    -1   -1   0
+$EndComp
+$Comp
+L Jumper:SolderJumper_2_Open JP3
+U 1 1 609FF8D2
+P 3150 6850
+F 0 "JP3" H 3150 6963 50  0000 C CNN
+F 1 "SolderJumper_2_Open" H 3150 6964 50  0001 C CNN
+F 2 "Jumper:SolderJumper-2_P1.3mm_Open_RoundedPad1.0x1.5mm" H 3150 6850 50  0001 C CNN
+F 3 "~" H 3150 6850 50  0001 C CNN
+	1    3150 6850
+	1    0    0    -1
+$EndComp
+Wire Wire Line
+	3100 6650 3100 6550
+Wire Wire Line
+	2800 6650 2900 6650
+Wire Wire Line
+	3200 6550 3200 6650
+Wire Wire Line
+	3200 6650 3400 6650
+Wire Wire Line
+	3300 6850 3400 6850
+Wire Wire Line
+	3400 6850 3400 6650
+Connection ~ 3400 6650
+Wire Wire Line
+	3400 6650 3550 6650
+Wire Wire Line
+	3000 6850 2900 6850
+Wire Wire Line
+	2900 6850 2900 6650
+Connection ~ 2900 6650
+Wire Wire Line
+	2900 6650 3100 6650
+$Comp
+L Device:C C2
+U 1 1 60A38D35
+P 1800 6650
+F 0 "C2" H 1915 6696 50  0000 L CNN
+F 1 "100nF" H 1915 6605 50  0000 L CNN
+F 2 "Capacitor_SMD:C_0805_2012Metric" H 1838 6500 50  0001 C CNN
+F 3 "~" H 1800 6650 50  0001 C CNN
+F 4 "C49678" H 1800 6650 50  0001 C CNN "LCSC"
+	1    1800 6650
+	1    0    0    -1
+$EndComp
+Wire Wire Line
+	1800 6500 1800 6200
+Wire Wire Line
+	1800 6200 2500 6200
+Connection ~ 2500 6200
+Wire Wire Line
+	2500 6200 2500 6100
+Wire Wire Line
+	1800 6800 1800 7100
+Wire Wire Line
+	1800 7100 2500 7100
+Connection ~ 2500 7100
+Wire Wire Line
+	2500 7100 2500 7200
+NoConn ~ 3600 2950
 Wire Bus Line
 	4200 2650 4200 5300
 Wire Bus Line
+	1800 2650 1800 5300
+Wire Bus Line
 	6900 2650 6900 5300
-Wire Bus Line
-	1800 2650 1800 5300
 $EndSCHEMATC
