File: Hardware/Serial Card/Serial Card.kicad_sch (KiCad schematic)
At the start: 35 parts, among them J1 Conn_02x08_Odd_Even, J2 DB9_Female, J3 Conn_01x03, P1 USB_C_Plug_USB2.0, U1 74LS138, U2 MAX238, U3 74HC02, U4 R65C52, U5 FT232RL, Y1 1.8432 Mhz

Commit message: Cleanup
Parts:
- C1, C2, C3, C4, C5: symbol Serial Card-rescue:CP-Device -> Serial_Card:CP-Device
- J2: symbol Serial Card-rescue:DB9_Female-Connector -> Serial_Card:DB9_Female-Connector

Commit message: Cleanup
Connections:
- net R~{W} renamed RWB
- net RWB: now also CONN1.RWB; no longer CONN1.R~{W}
- net ~{IRQ} renamed IRQB
- net IRQB: now also CONN1.IRQB; no longer CONN1.~{IRQ}
- net ~{NMI} renamed NMIB
- net NMIB: now also CONN1.NMIB; no longer CONN1.~{NMI}
- net ~{RES} renamed RESB
- net RESB: now also CONN1.RESB; no longer CONN1.~{RES}
Changed lines of the file:
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@@
 		)
 	)
-	(label "~{RES}"
+	(label "RESB"
 		(at 27.94 31.75 0)
 		(fields_autoplaced yes)
@@
 		)
 	)
-	(label "R~{W}"
+	(label "RWB"
 		(at 27.94 119.38 0)
 		(fields_autoplaced yes)
@@
 		)
 	)
-	(label "~{NMI}"
+	(label "NMIB"
 		(at 27.94 36.83 0)
 		(fields_autoplaced yes)
@@
 		)
 	)
-	(label "R~{W}"
+	(label "RWB"
 		(at 27.94 44.45 0)
 		(fields_autoplaced yes)
@@
 		)
 	)
-	(label "~{RES}"
+	(label "RESB"
 		(at 27.94 124.46 0)
 		(fields_autoplaced yes)
@@
 		)
 	)
-	(label "~{IRQ}"
+	(label "IRQB"
 		(at 27.94 34.29 0)
 		(fields_autoplaced yes)
@@
 		)
 	)
-	(global_label "~{RES}"
+	(global_label "RESB"
 		(shape input)
 		(at 185.42 134.62 180)
@@
 		)
 	)
-	(global_label "~{IRQ}"
+	(global_label "IRQB"
 		(shape output)
 		(at 144.78 77.47 90)
@@
 		)
 	)
-	(global_label "~{NMI}"
+	(global_label "NMIB"
 		(shape output)
 		(at 144.78 90.17 270)
@@
 		(pin "RDY"
 		)
-		(pin "R~{W}"
+		(pin "IRQB"
 		)
 		(pin "VCC"
@@
 		(pin "VCC"
 		)
-		(pin "~{IRQ}"
-		)
-		(pin "~{ML}"
-		)
-		(pin "~{NMI}"
-		)
-		(pin "~{RES}"
+		(pin "MLB"
+		)
+		(pin "NMIB"
+		)
+		(pin "RESB"
+		)
+		(pin "RWB"
 		)
 		(instances

Commit message: Updates
Parts:
- removed P1: USB_C_Plug_USB2.0, Connector_USB:USB_C_Receptacle_HRO_TYPE-C-31-M-12, symbol Serial_Card:USB_C_Plug_USB2.0
- added J4: USB_C_Receptacle_USB2.0, Connector_USB:USB_C_Receptacle_HRO_TYPE-C-31-M-12, symbol Connector:USB_C_Receptacle_USB2.0_16P
- C1, C2, C3, C4, C5: symbol Serial_Card:CP-Device -> Device:C_Polarized
- D1: value B5819W -> 1N5819; footprint Diode_SMD:D_SOD-123 -> Diode_SMD:D_SOD-323F; symbol Device:D_Schottky -> Diode:1N5819; LCSC C8598 -> C191023
Connections:
- net GND: now also J4.A1 (GND), J4.A12 (GND), J4.B1 (GND), J4.B12 (GND), J4.S1 (SHIELD)
- net at D1.2 (A): now also J4.A4 (VBUS), J4.A9 (VBUS), J4.B4 (VBUS), J4.B9 (VBUS)
- net at R6.1: now also J4.A5 (CC1)
- net at C10.2, R2.2: now also J4.A7 (D-), J4.B7 (D-)
- net at C9.2, R1.2: now also J4.A6 (D+), J4.B6 (D+)
- net at R5.1: now also J4.B5 (CC2)
- no-connect marks 27 -> 29

Commit message: Working on new PCBs
Parts:
- removed C1, C2, C3, C4, C5: 1uF, Capacitor_SMD:C_1206_3216Metric, symbol Device:C_Polarized
- removed C10, C9: 47pF, Capacitor_SMD:C_0805_2012Metric, symbol Device:C
- removed C11, C12, C13, C14, C15: 100nF, Capacitor_SMD:C_0805_2012Metric, symbol Device:C
- removed D1: 1N5819, Diode_SMD:D_SOD-323F, symbol Diode:1N5819
- removed D2, D3: LED, LED_SMD:LED_0805_2012Metric, symbol Device:LED
- removed J3: Conn_01x03, Connector_PinHeader_2.54mm:PinHeader_1x03_P2.54mm_Vertical, symbol Connector_Generic:Conn_01x03
- removed J4: USB_C_Receptacle_USB2.0, Connector_USB:USB_C_Receptacle_HRO_TYPE-C-31-M-12, symbol Connector:USB_C_Receptacle_USB2.0_16P
- removed R2: 27, Resistor_SMD:R_0805_2012Metric, symbol Device:R
- removed R3, R4: 330, Resistor_SMD:R_0805_2012Metric, symbol Device:R
- removed R5, R6: 5.1k, Resistor_SMD:R_0805_2012Metric, symbol Device:R
- removed U2: MAX238, Package_SO:SOIC-24W_7.5x15.4mm_P1.27mm, symbol Serial_Card:MAX238
- removed U3: 74HC02, Package_SO:SO-14_3.9x8.65mm_P1.27mm, symbol 74xx:74HC02
- removed U4: R65C52, Package_DIP:DIP-40_W15.24mm_Socket, symbol Serial_Card:R65C52
- removed U5: FT232RL, Package_SO:SSOP-28_5.3x10.2mm_P0.65mm, symbol Serial_Card:FT232RL
- added C1, C5: 100nF, Capacitor_SMD:C_0805_2012Metric, symbol Device:C
- added C3, C6, C7: 1uF, Capacitor_SMD:C_0805_2012Metric, symbol Device:C
- added U1: 65C51, Package_DIP:DIP-28_W15.24mm_Socket_LongPads, symbol 6502 Parts:65C51
- added U2: MAX232, Package_SO:SOIC-16W_5.3x10.2mm_P1.27mm, symbol Interface_UART:MAX232
- C8: value 22pF -> 1uF; LCSC C1804 -> C28323
- J1: renamed from CONN1; footprint Serial Card:6502CARDEDGE -> 6502 Parts:6502CARDEDGE; symbol Serial_Card:6502CARDEDGE -> 6502 Parts:6502CARDEDGE
- J3: renamed from J2; footprint Serial Card:DB9 -> 6502 Parts:DB9; symbol Serial_Card:DB9_Female-Connector -> 6502 Parts:DB9
- R1: value 27 -> 1M; LCSC C17594 -> C103906
- renumbered C7 to C2, C6 to C4, J1 to J2, U1 to U3
Connections:
- net A0: now also U1.13 (RS0)
- net A1: now also U1.14 (RS1)
- net D0: now also U1.18 (D0)
- net D1: now also U1.19 (D1)
- net D2: now also U1.20 (D2)
- net D3: now also U1.21 (D3)
- net D4: now also U1.22 (D4)
- net D5: now also U1.23 (D5)
- net D6: now also U1.24 (D6)
- net D7: now also U1.25 (D7)
- net GND: now also C8.2, R1.1, Y1.2, C1.2, C5.2, C7.2, U1.1 (GND), U1.7 (XTALO), U2.15 (GND); no longer C8.1
- net IRQB: now also U1.26 (IRQB)
- net RESB: now also U1.4 (RESB)
- net RWB: now also U1.28 (RWB)
- net VCC: now also C1.1, C5.1, U1.15 (VCC), U1.2 (CS0), U2.16 (VCC)
- net PHI2: now reaches J1.PHI2
- net PHI2: now also U1.27 (PHI2)
- net at C2.2, Y1.1: now also R1.2, U1.6 (XTALI)
- net A2: no longer names the net of J1.A2
- net CTS: no longer names the net of J3.8
- net DCD: no longer names the net of J3.1
- net DSR: no longer names the net of J3.6
- net DTR: no longer names the net of J3.4
- net NMIB: no longer names the net of J1.NMIB
- net RTS: no longer names the net of J3.7
- net RX: no longer names the net of J3.2
- net RX: now also U2.14 (T1OUT)
- net TX: no longer names the net of J3.3
- net TX: now also U2.13 (R1IN)
- net ~{CS} renamed CSB
- net CSB: now also U1.3 (CS1B)
- new net: C8.1, U2.6 (VS-)
- new net: C7.1, U2.2 (VS+)
- new net: C6.1, U2.4 (C2+)
- new net: C6.2, U2.5 (C2-)
- new net: C3.1, U2.1 (C1+)
- new net: C3.2, U2.3 (C1-)
- new net R1OUT: U1.12 (RXD), U2.12 (R1OUT)
- new net T1IN: U1.10 (TXD), U2.11 (T1IN)
- no-connect marks 29 -> 32
Other:
- moved on the sheet: C2, C4, J1, J2, J3, U3, Y1

Commit message: Pi Card PCB
Parts:
- removed C7: 1uF, Capacitor_SMD:C_0805_2012Metric, symbol Device:C
- removed U2: MAX232, Package_SO:SOIC-16W_5.3x10.2mm_P1.27mm, symbol Interface_UART:MAX232
- added C4: 1uF, Capacitor_SMD:C_0805_2012Metric, symbol Device:C
- added U2: MAX238, Package_DIP:DIP-24_W7.62mm_Socket_LongPads, symbol 6502 Parts:MAX238
- renumbered C4 to C7
Connections:
- net GND: now also C5.1, U2.8 (GND); no longer C5.2
- net VCC: now also C5.2, C6.1, U2.9 (VCC); no longer C5.1
- net DCD: now reaches J3.1
- net DCD: now also U2.16 (R4IN)
- net RXD: now reaches J3.2
- net RXD: now also U2.7 (R1IN)
- net TXD: now reaches J3.3
- net TXD: now also U2.2 (T1OUT)
- net DTR: now reaches J3.4
- net DTR: now also U2.1 (T2OUT)
- net DSR: now reaches J3.6
- net DSR: now also U2.23 (R3IN)
- net RTS: now reaches J3.7
- net RTS: now also U2.24 (T3OUT)
- net CTS: now reaches J3.8
- net CTS: now also U2.3 (R2IN)
- net at C8.1: now also U2.15 (V-)
- net at C6.2: now also U2.11 (V+)
- net DTROUT: now reaches U1.11 (DTRB)
- net DTROUT: now also U2.18 (T2IN)
- net DCDIN: now reaches U1.16 (DCDB)
- net DCDIN: now also U2.17 (R4OUT)
- net DSRIN: now reaches U1.17 (DSRB)
- net DSRIN: now also U2.22 (R3OUT)
- net RTSOUT: now reaches U1.8 (RTSB)
- net RTSOUT: now also U2.19 (T3IN)
- net CTSIN: now reaches U1.9 (CTSB)
- net CTSIN: now also U2.4 (R2OUT)
- net at C3.1: now also U2.10 (C1+)
- net at C3.2: now also U2.12 (C1-)
- net R1OUT renamed RXDIN
- net RXDIN: now also U2.6 (R1OUT)
- net T1IN renamed TXDOUT
- net TXDOUT: now also U2.5 (T1IN)
- new net: C4.1, U2.13 (C2+)
- new net: C4.2, U2.14 (C2-)
- no-connect marks 32 -> 20
Other:
- moved on the sheet: J3

Commit message: Add production files
Parts:
- J1, J2, J3, U1, U2, Y1: now left out of the parts list
Changed lines of the file:
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@@
 		(unit 1)
 		(exclude_from_sim no)
-		(in_bom yes)
+		(in_bom no)
 		(on_board yes)
 		(dnp no)
@@
 		(unit 1)
 		(exclude_from_sim no)
-		(in_bom yes)
+		(in_bom no)
 		(on_board yes)
 		(dnp no)
@@
 		(unit 1)
 		(exclude_from_sim no)
-		(in_bom yes)
+		(in_bom no)
 		(on_board yes)
 		(dnp no)
@@
 		(unit 1)
 		(exclude_from_sim no)
-		(in_bom yes)
+		(in_bom no)
 		(on_board yes)
 		(dnp no)
@@
 		(unit 1)
 		(exclude_from_sim no)
-		(in_bom yes)
+		(in_bom no)
 		(on_board yes)
 		(dnp no)
@@
 		(unit 1)
 		(exclude_from_sim no)
-		(in_bom yes)
-		(on_board yes)
-		(dnp no)
+		(in_bom no)
+		(on_board yes)
+		(dnp no)

Commit message: Add LCD Card
Parts:
- added D1: D_Schottky, Diode_THT:D_DO-35_SOD27_P7.62mm_Horizontal, symbol Device:D_Schottky
- added JP1: SolderJumper_2_Bridged, Jumper:SolderJumper-2_P1.3mm_Bridged_RoundedPad1.0x1.5mm, symbol Jumper:SolderJumper_2_Bridged
Connections:
- net IRQB: now also D1.2 (A), JP1.1 (A); no longer U1.26 (IRQB)
- new net: D1.1 (K), JP1.2 (B), U1.26 (IRQB)
Other:
- moved on the sheet: C1, C2, R1, U1, Y1
