File: Hardware/Giga Shield/Giga Shield.kicad_pcb (KiCad board)
At the start: 2 copper layers, 101.6 x 53.3 mm, 27 parts, among them J1 Conn_02x20_Odd_Even, U1 TXS0108EPW, U2 TXS0108EPW, U3 TXS0108EPW, U4 TXS0108EPW, U5 TXS0108EPW

Commit message: Cleanup
Parts:
- A1: footprint 6502 Parts:Arduino_Giga_R1_WiFi_Shield -> 6502 Parts:Arduino Giga R1 WiFi Shield
- J1: value Conn_02x20_Odd_Even -> 6502 Bus
