File: Hardware/Giga Shield/Giga Shield.kicad_sch (KiCad schematic)
At the start: 24 parts, among them J1 Conn_02x20_Odd_Even, U1 TXS0108EPW, U2 TXS0108EPW, U3 TXS0108EPW, U4 TXS0108EPW, U5 TXS0108EPW

Commit message: Cleanup
Parts:
- A1: footprint 6502 Parts:Arduino_Giga_R1_WiFi_Shield -> 6502 Parts:Arduino Giga R1 WiFi Shield
- J1: value Conn_02x20_Odd_Even -> 6502 Bus
Changed lines of the file:
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@@
 	(title_block
 		(title "6502 Giga Shield")
-		(date "2024-04-08")
+		(date "2024-06-12")
 		(rev "1.0")
 		(company "A.C. Wright Design")
@@
 			)
 		)
-		(property "Footprint" "6502 Parts:Arduino_Giga_R1_WiFi_Shield"
+		(property "Footprint" "6502 Parts:Arduino Giga R1 WiFi Shield"
 			(at 203.2 163.83 0)
 			(effects
@@
 		(dnp no)
 		(property "Reference" "C12"
-			(at 74.93 189.1792 90)
+			(at 74.93 199.6186 90)
 			(effects
 				(font
@@
 		)
 		(property "Value" "100nF"
-			(at 74.93 191.4906 90)
+			(at 74.93 201.93 90)
 			(effects
 				(font
@@
 			)
 		)
-		(property "Value" "Conn_02x20_Odd_Even"
-			(at 74.93 135.2296 0)
+		(property "Value" "6502 Bus"
+			(at 74.93 189.992 0)
 			(effects
 				(font
 					(size 1.27 1.27)
 				)
-				(hide yes)
 			)
 		)
