File: Hardware/Memory Card/Memory Card.kicad_pcb (KiCad board)
At the start: 2 copper layers, 100 x 57.6 mm, 21 parts, among them IC1 AS6C62256, IC2 AT28C256, J1 Conn_02x01, J2 Conn_02x02_Odd_Even, U1 74HC00, U2 74HC00, U3 74HC00

Commit message: Cleanup
Routing:
- net GND: vias 3 -> 19
Other:
- board text added: "© 2024 A.C. Wright Design | acwrightdesign.com | Rev 2.0"
- board text removed: "© 2021 A.C. Wright Design | acwrightdesign.com | Rev 1.1"

Commit message: Cleanup
Parts:
- CONN1: value 6502CARDEDGECONNECTOR -> 6502CARDEDGE
Connections:
- CONN1 pad BE: Net-(CONN1-PadBE) -> unconnected-(CONN1-PadBE)
- CONN1 pad EXP2: (no net) -> unconnected-(CONN1-PadEXP2)
- CONN1 pad EXP3: (no net) -> unconnected-(CONN1-PadEXP3)
- CONN1 pad RDY: Net-(CONN1-PadRDY) -> unconnected-(CONN1-PadRDY)
- U1 pad 1: R~{W} -> RWB
- U1 pad 10: R~{W} -> RWB
- U1 pad 9: R~{W} -> RWB
Routing:
- net R~{W}: track 59.4 -> 0.00 mm, vias 2 -> 0
- net RWB: track 0.00 -> 59.4 mm, vias 0 -> 2

Commit message: Updates
Parts:
- added TP1: ~{ROM_ENABLE}, TestPoint:TestPoint_Pad_1.0x1.0mm, F.Cu at (191.5, 100.2)
- added TP2: ~{HI_ROM_DISABLE}, TestPoint:TestPoint_Pad_1.0x1.0mm, F.Cu at (109.1, 84.0)
- added TP3: ~{READ}, TestPoint:TestPoint_Pad_1.0x1.0mm, F.Cu at (189.1, 114.4)
- added TP4: ~{WRITE}, TestPoint:TestPoint_Pad_1.0x1.0mm, F.Cu at (180.7, 122.2)
- added TP5: GND, TestPoint:TestPoint_Pad_1.0x1.0mm, F.Cu at (191.4, 94.8)
Routing:
- net ~{ROM_ENABLE}: track 68.2 -> 94.5 mm, vias 2 -> 4
- net ~{READ}: track 80.9 -> 99.1 mm, vias 4 -> 5
- net ~{HI_ROM_DISABLE}: track 78.4 -> 83.4 mm
- net ~{WRITE}: track 90.3 -> 93.0 mm
- net VCC: track 262.0 -> 261.3 mm

Commit message: Working on new PCBs
Parts:
- G***: footprint 6502 Logo:6502 Logo 5mm -> 6502 Logos:6502 Memory Card Logo 5mm
- J1: renamed from CONN1; footprint Memory Card:6502CARDEDGE -> 6502 Parts:6502CARDEDGE
- moved TP3 0.14 mm to (191.5, 94.9)
- renumbered J1 to J3, JP2 to JP1, JP3 to JP2, JP1 to JP3, R2 to R1, R1 to R2, TP2 to TP1, TP1 to TP2, TP5 to TP3, TP3 to TP4, TP4 to TP5, U3 to U1, IC1 to U3, IC2 to U4, U1 to U5
Connections:
- net ~{HI_ROM_DISABLE} renamed HRDB
- net ~{READ} renamed RB
- net ~{ROM_ENABLE} renamed REB
- net ~{WRITE} renamed WB
Other:
- board text added: "~{HI ROM DIS}"
- board text added: "© 2024 A.C. Wright Design | acwrightdesign.com | Rev 1.0"
- board text removed: "~{HI} ROM DIS"
- board text removed: "© 2024 A.C. Wright Design | acwrightdesign.com | Rev 2.0"

Commit message: Pi Card PCB
Parts:
- moved G*** 90.7 mm to (103.0, 121.7)
- moved REF** 17.5 mm to (192.2, 121.1)
- moved G*** 0.69 mm to (102.9, 98.9)

Commit message: Cleanup
Parts:
- J1: value 6502CARDEDGE -> 6502 Card Edge; footprint 6502 Parts:6502CARDEDGE -> 6502 Parts:6502 Card Edge
