File: Templates/Card/Card.kicad_sch (KiCad schematic)
At the start: 4 parts, among them J1 6502 Bus, J2 Conn_02x08_Odd_Even, U1 74HC138

Commit message: Add sound card
Parts:
- J1: value 6502 Bus -> 6502 Card Edge; symbol 6502 Parts:6502 Bus -> 6502 Parts:6502 Card Edge
Changed lines of the file:
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@@
 	)
 	(symbol
-		(lib_id "6502 Parts:6502 Bus")
+		(lib_id "6502 Parts:6502 Card Edge")
 		(at 71.12 62.23 0)
 		(unit 1)
@@
 		(dnp no)
 		(property "Reference" "J1"
-			(at 60.96 33.782 0)
+			(at 60.706 33.528 0)
 			(effects
 				(font
@@
 			)
 		)
-		(property "Value" "6502 Bus"
-			(at 65.532 35.306 0)
+		(property "Value" "6502 Card Edge"
+			(at 68.58 35.052 0)
 			(effects
 				(font
