File: Hardware/GPIO Card/GPIO Card.kicad_sch (KiCad schematic)
At the start: 10 parts, among them J1 6502CARDEDGE, J2 Conn_02x08_Odd_Even, J3 PORT A, J4 PORT B, U1 74HC138, U2 65C22

Commit message: Production updates
Parts:
- J3, J4: now left out of the parts list
Changed lines of the file:
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@@
 		(unit 1)
 		(exclude_from_sim no)
-		(in_bom yes)
+		(in_bom no)
 		(on_board yes)
 		(dnp no)
@@
 		(unit 1)
 		(exclude_from_sim no)
-		(in_bom yes)
+		(in_bom no)
 		(on_board yes)
 		(dnp no)

Commit message: Cleanup
Parts:
- J1: value 6502CARDEDGE -> 6502 Card Edge; footprint 6502 Parts:6502CARDEDGE -> 6502 Parts:6502 Card Edge; symbol 6502 Parts:6502CARDEDGE -> 6502 Parts:6502 Card Edge

Commit message: Revise some boards
Parts:
- J3, J4: footprint Connector_PinHeader_2.54mm:PinHeader_2x06_P2.54mm_Vertical -> 6502 Parts:6502 GPIO Connector
Changed lines of the file:
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@@
 			)
 		)
-		(property "Footprint" "Connector_PinHeader_2.54mm:PinHeader_2x06_P2.54mm_Vertical"
+		(property "Footprint" "6502 Parts:6502 GPIO Connector"
 			(at 226.06 69.85 0)
 			(effects
@@
 			)
 		)
-		(property "Footprint" "Connector_PinHeader_2.54mm:PinHeader_2x06_P2.54mm_Vertical"
+		(property "Footprint" "6502 Parts:6502 GPIO Connector"
 			(at 226.06 43.18 0)
 			(effects
