File: Hardware/GPIO Helper/GPIO Helper.kicad_sch (KiCad schematic)
At the start: 34 parts, among them J1 PORT A, J2 PORT B, SW1 PA7, SW2 PA6, SW3 PA5, SW4 PA4, SW5 PA3, SW6 PA2, SW7 PA1, SW8 PA0

Commit message: Revise some boards
Parts:
- J1, J2: footprint Connector_PinHeader_2.54mm:PinHeader_2x06_P2.54mm_Vertical -> 6502 Parts:6502 GPIO Connector
Changed lines of the file:
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@@
 			)
 		)
-		(property "Footprint" "Connector_PinHeader_2.54mm:PinHeader_2x06_P2.54mm_Vertical"
+		(property "Footprint" "6502 Parts:6502 GPIO Connector"
 			(at 203.2 50.8 0)
 			(effects
@@
 			)
 		)
-		(property "Footprint" "Connector_PinHeader_2.54mm:PinHeader_2x06_P2.54mm_Vertical"
+		(property "Footprint" "6502 Parts:6502 GPIO Connector"
 			(at 82.55 50.8 0)
 			(effects
