File: Hardware/Storage Card/Storage Card.kicad_pcb (KiCad board)
At the start: 2 copper layers, 100 x 57.6 mm, 7 parts, among them J1 6502 Card Edge, J2 Conn_02x08_Odd_Even, U1 74HC138

Commit message: More PCBs
Parts:
- added C2: 100nF, Capacitor_SMD:C_0805_2012Metric, F.Cu at (126.5, 94.7)
- added D1: ACT, LED_SMD:LED_0805_2012Metric, F.Cu at (125.0, 86.1)
- added J3: Compact Flash, 6502 Parts:SD-SMD_CFH-L3C1LBL01MN0, F.Cu at (169.0, 108.5)
- added J4: ACT LED, Connector_JST:JST_XH_B2B-XH-A_1x02_P2.50mm_Vertical, F.Cu at (127.0, 77.0)
- added R1: 1k, Resistor_SMD:R_0805_2012Metric, F.Cu at (140.7, 83.6)
- added R2: 1k, Resistor_SMD:R_0805_2012Metric, F.Cu at (140.7, 80.7)
- added R3: 1k, Resistor_SMD:R_0805_2012Metric, F.Cu at (140.7, 77.9)
- added R4: 1k, Resistor_SMD:R_0805_2012Metric, F.Cu at (140.7, 75.0)
- added R5: 330, Resistor_SMD:R_0805_2012Metric, F.Cu at (131.6, 86.1)
- added R6: 330, Resistor_SMD:R_0805_2012Metric, F.Cu at (128.3, 86.1)
- added U1: 74HC00, Package_SO:SOIC-14_3.9x8.7mm_P1.27mm, F.Cu at (133.5, 97.5)
- moved G*** 0.14 mm to (195.0, 115.0)
- renumbered U1 to U2
Connections:
- J1 pad A3: A3 -> unconnected-(J1-PadA3)
- J1 pad IRQB: IRQB -> unconnected-(J1-PadIRQB)
Routing:
- net CSB: track 26.5 -> 101.4 mm
- net VCC: track 102.9 -> 172.1 mm, vias 6 -> 10
- net Net-(J3-~{CS1}): track 0.00 -> 64.6 mm, vias 0 -> 2
- net Net-(J3-~{WE}): track 0.00 -> 62.5 mm, vias 0 -> 2
- net Net-(J3-~{DASP}): track 0.00 -> 58.0 mm, vias 0 -> 2
- net Net-(J3-~{PDIAG}): track 0.00 -> 55.4 mm, vias 0 -> 2
- net ~{RD}: track 0.00 -> 55.3 mm, vias 0 -> 2
- net Net-(J3-~{REG}): track 0.00 -> 55.0 mm, vias 0 -> 2
- net ~{WR}: track 0.00 -> 53.7 mm, vias 0 -> 2
- net RESB: track 12.5 -> 56.8 mm, vias 1 -> 2
- net D7: track 0.00 -> 43.8 mm, vias 0 -> 2
- net D6: track 0.00 -> 42.4 mm, vias 0 -> 2
- net D5: track 0.00 -> 41.0 mm, vias 0 -> 2
- net D4: track 0.00 -> 39.9 mm, vias 0 -> 2
- net D3: track 0.00 -> 38.3 mm, vias 0 -> 2
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Other:
- board text added: "+"
- board text added: "K"
