File: Hardware/Storage Card/Storage Card.kicad_sch (KiCad schematic)
At the start: 5 parts, among them J1 6502 Card Edge, J2 Conn_02x08_Odd_Even, J3 Compact Flash, U1 74HC138

Commit message: More PCBs
Parts:
- added C2: 100nF, Capacitor_SMD:C_0805_2012Metric, symbol Device:C
- added D1: ACT, LED_SMD:LED_0805_2012Metric, symbol Device:LED
- added J4: ACT LED, Connector_JST:JST_XH_B2B-XH-A_1x02_P2.50mm_Vertical, symbol Connector_Generic:Conn_01x02
- added R1, R2, R3, R4: 1k, Resistor_SMD:R_0805_2012Metric, symbol Device:R
- added R5, R6: 330, Resistor_SMD:R_0805_2012Metric, symbol Device:R
- added U1: 74HC00, Package_SO:SOIC-14_3.9x8.7mm_P1.27mm, symbol 74xx:74HC00
- J3: footprint (none) -> 6502 Parts:SD-SMD_CFH-L3C1LBL01MN0; LCSC (none) -> C444350
- renumbered U1 to U2
Connections:
- net A0: now also J3.20 (A0)
- net A1: now also J3.19 (A1)
- net A2: now also J3.18 (A2)
- net CSB: now also J3.7 (~{CS0})
- net D0: now also J3.21 (D0)
- net D1: now also J3.22 (D1)
- net D2: now also J3.23 (D2)
- net D3: now also J3.2 (D3)
- net D4: now also J3.3 (D4)
- net D5: now also J3.4 (D5)
- net D6: now also J3.5 (D6)
- net D7: now also J3.6 (D7)
- net GND: now also J3.1 (GND), J3.10 (A9), J3.11 (A8), J3.12 (A7), J3.14 (A6), J3.15 (A5), J3.16 (A4), J3.17 (A3), J3.39 (~{CSEL}), J3.50 (GND), J3.8 (A10), J3.9 (~{ATA_SEL}), C2.2, U1.12, U1.13, U1.7 (GND)
- net PHI2: now also U1.10, U1.5
- net RESB: now also J3.41 (~{RESET})
- net RWB: now also U1.1, U1.2, U1.4
- net VCC: now also J3.13 (VCC), J3.38 (VCC), C2.1, D1.2 (A), J4.1 (Pin_1), R1.2, R2.2, R3.1, R4.1, U1.14 (VCC)
- net at J3.32 (~{CS1}): now also R1.1
- net ~{RD}: now reaches J3.34 (~{IORD})
- net ~{RD}: now also U1.6
- net ~{WR}: now reaches J3.35 (~{IOWR})
- net ~{WR}: now also U1.8
- net at J3.36 (~{WE}): now also R2.1
- net at J3.44 (~{REG}): now also R3.2
- net at J3.45 (~{DASP}): now also R5.1, R6.1
- net at J3.46 (~{PDIAG}): now also R4.2
- net A3: no longer names the net of J1.A3
- net IRQB: no longer names the net of J1.IRQB
- new net: J4.2 (Pin_2), R6.2
- new net: U1.3, U1.9
- new net: D1.1 (K), R5.2
- no-connect marks 14 -> 32
Other:
- note removed: "Needs to be changed to True IDE pinout"
