File: Hardware/Teensy Card/Teensy Card.kicad_pcb (KiCad board)
At the start: 2 copper layers, 100 x 57.6 mm, 14 parts, among them J1 6502 Card Edge, U1 Teensy4.1, U2 SN74LVC4245APWR, U3 SN74LVC4245APWR, U4 SN74LVC4245APWR, U5 SN74LVC4245APWR, U6 SN74LVC4245APWR

Commit message: Keypad and Teensy boards
Parts:
- added C1: 100nF, Capacitor_SMD:C_0805_2012Metric, F.Cu at (172.5, 105.3)
- added C2: 100nF, Capacitor_SMD:C_0805_2012Metric, F.Cu at (157.0, 105.3)
- added C3: 100nF, Capacitor_SMD:C_0805_2012Metric, F.Cu at (140.9, 105.3)
- added C4: 100nF, Capacitor_SMD:C_0805_2012Metric, F.Cu at (126.0, 84.3)
- added C5: 100nF, Capacitor_SMD:C_0805_2012Metric, F.Cu at (126.0, 105.3)
- added J1: GPIO, 6502 Parts:6502 GPIO Connector, F.Cu at (189.8, 105.8)
- added R5: 1k, Resistor_SMD:R_0805_2012Metric, F.Cu at (128.1, 116.8)
- added SW1: A Select, 6502 Parts:DS01C-254-L-08BE, F.Cu at (113.6, 89.7)
- added SW2: B Select, 6502 Parts:DS01C-254-L-08BE, F.Cu at (113.7, 112.7)
- U6: renamed from U1; footprint Teensy:Teensy41 -> Teensy:Teensy41 Basic
- moved U1 105.2 mm to (174.7, 111.6)
- moved R1 102.6 mm to (174.7, 116.8)
- moved R2 87.8 mm to (159.2, 116.8)
- moved U2 85.0 mm to (159.2, 111.6)
- moved U3 73.1 mm to (143.1, 111.6)
- moved R4 71.1 mm to (143.2, 116.7)
- moved REF** 67.9 mm to (178.4, 121.8)
- moved U5 51.0 mm to (128.2, 111.6)
- moved U4 50.4 mm to (128.2, 90.6)
- moved R3 48.9 mm to (128.1, 95.9)
- moved U6 1.06 mm to (167.8, 90.2)
- renumbered J1 to J2, U2 to U1, U4 to U2, U5 to U4, U6 to U5
Connections:
- R1 pad 1: Net-(U5-A7) -> VCC
- R1 pad 2: GND -> OE1
- R2 pad 1: Net-(U5-B7) -> VCC
- R2 pad 2: GND -> OE3
- R3 pad 1: Net-(U6-A3) -> VCC
- R3 pad 2: GND -> OE4
- R4 pad 1: Net-(U6-B3) -> VCC
- R4 pad 2: GND -> OE2
- U4 pad 10: Net-(U5-A7) -> SYNC_A
- U4 pad 14: Net-(U5-B7) -> SYNC_3V3
- U4 pad 15: Net-(U5-B7) -> RWB_3V3
- U4 pad 3: PHI2 -> PHI2_A
- U4 pad 4: BE -> BE_A
- U4 pad 5: RDY -> RDY_A
- U4 pad 6: NMIB -> NMIB_A
- U4 pad 7: IRQB -> IRQB_A
- U4 pad 8: RESB -> RESB_A
- U4 pad 9: Net-(U5-A7) -> RWB_A
- U5 pad 10: Net-(U6-A3) -> SYNC_B
- U5 pad 14: Net-(U6-B3) -> RWB_3V3
- U5 pad 15: Net-(U6-B3) -> RWB_3V3
- U5 pad 16: Net-(U6-B3) -> RESB_3V3
- U5 pad 17: Net-(U6-B3) -> IRQB_3V3
- U5 pad 18: Net-(U6-B3) -> NMIB_3V3
- U5 pad 19: Net-(U6-B3) -> RDY_3V3
- U5 pad 20: SYNC_3V3 -> BE_3V3
- U5 pad 21: RWB_3V3 -> PHI2_3V3
- U5 pad 3: RWB -> PHI2_B
- U5 pad 4: SYNC -> BE_B
- U5 pad 5: Net-(U6-A3) -> RDY_B
- U5 pad 6: Net-(U6-A3) -> NMIB_B
- U5 pad 7: Net-(U6-A3) -> IRQB_B
- U5 pad 8: Net-(U6-A3) -> RESB_B
- U5 pad 9: Net-(U6-A3) -> RWB_B
- U6 pad 10: unconnected-(U1-8_TX2_IN1-Pad10) -> GPIO2
- U6 pad 11: unconnected-(U1-9_OUT1C-Pad11) -> GPIO3
- U6 pad 12: unconnected-(U1-10_CS_MQSR-Pad12) -> GPIO4
- U6 pad 13: unconnected-(U1-11_MOSI_CTX1-Pad13) -> GPIO5
- U6 pad 14: unconnected-(U1-12_MISO_MQSL-Pad14) -> GPIO6
- U6 pad 16: unconnected-(U1-24_A10_TX6_SCL2-Pad16) -> OE4
- U6 pad 17: unconnected-(U1-25_A11_RX6_SDA2-Pad17) -> DIR4
- U6 pad 2: unconnected-(U1-0_RX1_CRX2_CS1-Pad2) -> OE1
- U6 pad 20: unconnected-(U1-28_RX7-Pad20) -> OE5
- U6 pad 21: unconnected-(U1-29_TX7-Pad21) -> DIR5
- U6 pad 22: unconnected-(U1-30_CRX3-Pad22) -> BE_3V3
- U6 pad 23: unconnected-(U1-31_CTX3-Pad23) -> RDY_3V3
- U6 pad 24: unconnected-(U1-32_OUT1B-Pad24) -> SYNC_3V3
- U6 pad 25: unconnected-(U1-33_MCLK2-Pad25) -> RESB_3V3
- U6 pad 26: unconnected-(U1-34_RX8-Pad26) -> IRQB_3V3
- U6 pad 27: unconnected-(U1-35_TX8-Pad27) -> NMIB_3V3
- U6 pad 28: unconnected-(U1-36_CS-Pad28) -> RWB_3V3
- U6 pad 29: unconnected-(U1-37_CS-Pad29) -> PHI2_3V3
- U6 pad 3: unconnected-(U1-1_TX1_CTX2_MISO1-Pad3) -> DIR1
- U6 pad 35: unconnected-(U1-13_SCK_LED-Pad35) -> GPIO7
- U6 pad 4: unconnected-(U1-2_OUT2-Pad4) -> OE2
- U6 pad 5: unconnected-(U1-3_LRCLK2-Pad5) -> DIR2
- U6 pad 6: unconnected-(U1-4_BCLK2-Pad6) -> OE3
- U6 pad 7: unconnected-(U1-5_IN2-Pad7) -> DIR3
- U6 pad 8: unconnected-(U1-6_OUT1D-Pad8) -> GPIO0
- U6 pad 9: unconnected-(U1-7_RX2_OUT1A-Pad9) -> GPIO1
Routing:
- net VCC: track 0.00 -> 211.3 mm, vias 0 -> 8
- net 3V3: track 0.00 -> 154.2 mm, vias 0 -> 7
- net OE2: track 0.00 -> 79.1 mm, vias 0 -> 6
- net PHI2: track 0.00 -> 78.4 mm, vias 0 -> 4
- net DIR2: track 0.00 -> 73.9 mm, vias 0 -> 4
- net BE: track 0.00 -> 71.0 mm, vias 0 -> 4
- net RDY: track 0.09 -> 63.0 mm, vias 0 -> 4
- net SYNC: track 0.08 -> 62.2 mm, vias 0 -> 3
- net RWB: track 0.09 -> 61.7 mm, vias 0 -> 3
- net OE3: track 0.00 -> 58.8 mm, vias 0 -> 2
- net NMIB: track 0.00 -> 57.7 mm, vias 0 -> 4
- net IRQB: track 0.00 -> 56.2 mm, vias 0 -> 4
- net PHI2_3V3: track 0.00 -> 56.1 mm, vias 0 -> 4
- net A9_3V3: track 0.00 -> 56.0 mm, vias 0 -> 4
- net DIR3: track 0.00 -> 55.7 mm, vias 0 -> 2
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Other:
- board text added: "0"
- board text added: "1"
- board text added: "2"
- board text added: "3"
- board text added: "3V3"
- board text added: "4"
- board text added: "5"
- board text added: "6"
- board text added: "7"
- board text added: "GND"

Commit message: Fix Teensy card
Parts:
- U1, U2, U3, U4, U5: footprint Package_SO:TSSOP-24_4.4x6.5mm_P0.5mm -> Package_SO:TSSOP-24_4.4x7.8mm_P0.65mm
- moved R4 0.28 mm to (143.2, 117.0)
- moved R1 0.23 mm to (174.7, 117.0)
- moved R2 0.23 mm to (159.2, 117.0)
- moved R5 0.23 mm to (128.1, 117.0)
- moved R3 0.08 mm to (128.1, 96.0)
Connections:
- U5 pad 14: RWB_3V3 -> SYNC_3V3
Routing:
- net SYNC_3V3: track 22.7 -> 45.5 mm
- net DIR3: track 55.7 -> 53.8 mm
- net 3V3: track 154.2 -> 155.6 mm
- net PHI2_B: track 11.2 -> 10.1 mm
- net AD6_3V3: track 39.7 -> 38.9 mm
- net PHI2: track 78.4 -> 79.2 mm
- net IRQB_3V3: track 37.7 -> 38.4 mm
- net RWB_3V3: track 42.4 -> 41.7 mm
- net DIR2: track 73.9 -> 74.6 mm
- net DIR1: track 48.9 -> 48.2 mm
- net AD7_3V3: track 45.4 -> 44.8 mm
- net A7: track 41.3 -> 40.8 mm
- net DIR4: track 35.3 -> 35.8 mm
- net OE5: track 52.8 -> 53.3 mm
- net D7: track 32.9 -> 32.4 mm
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