File: Hardware/LCD Card/Rev 1.1/LCD Card.kicad_sch (KiCad schematic)
At the start: 12 parts, among them J1 6502 Card Edge, J2 GPIO, J3 Conn_02x08_Odd_Even, U1 65C22, U2 LCD-16X2, U3 74HC138

Commit message: Update LCD trimpot part number and fix 3D model
Parts:
- VR1: footprint 6502 Parts:3386F-1-103TLF -> 6502 Parts:3386F-1-103LF
Changed lines of the file:
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@@
 			)
 		)
-		(property "Footprint" "6502 Parts:3386F-1-103TLF"
+		(property "Footprint" "6502 Parts:3386F-1-103LF"
 			(at 212.09 41.91 0)
 			(effects
