File: Hardware/Input Board/Rev 1.0/Input Board.kicad_sch (KiCad schematic)
At the start: 24 parts, among them J1 6502 Bus, J2 PORT B, J3 Conn_02x08_Odd_Even, J4 SNES Controller Port 1, J5 Keyboard, J6 Mouse, J7 SNES Controller Port 2, U1 65C22, U2 74HC138, U3 74HC595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

Commit message: Better 3D models and images
Parts:
- U4, U5: footprint Package_DIP:DIP-8_W7.62mm_LongPads -> Package_DIP:DIP-8_W7.62mm_Socket_LongPads
Changed lines of the file:
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@@
 			)
 		)
-		(property "Footprint" "Package_DIP:DIP-8_W7.62mm_LongPads"
+		(property "Footprint" "Package_DIP:DIP-8_W7.62mm_Socket_LongPads"
 			(at 193.04 41.91 0)
 			(effects
@@
 			)
 		)
-		(property "Footprint" "Package_DIP:DIP-8_W7.62mm_LongPads"
+		(property "Footprint" "Package_DIP:DIP-8_W7.62mm_Socket_LongPads"
 			(at 193.04 100.33 0)
 			(effects
