File: Hardware/Backplane Pro/Rev 1.0/Backplane Pro.kicad_pcb (KiCad board)
At the start: 2 copper layers, 100 x 100 mm, 49 parts, among them J1 PWR_SW, J10 Conn_02x20_Odd_Even, J2 USB_C_Receptacle_USB2.0, J3 RESET_SW, J4 CLOCK_ENBL_SW, J5 Conn_02x20_Odd_Even, J6 Conn_02x20_Odd_Even, J7 Conn_02x20_Odd_Even, J8 Conn_02x20_Odd_Even, J9 Conn_02x20_Odd_Even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

Commit message: Housekeeping
Parts:
- J10: value Conn_02x20_Odd_Even -> 6502 Bus
- J5, J6, J7, J8, J9: value Conn_02x20_Odd_Even -> 6502 Card Connector
