File: Hardware/Backplane/Rev 1.0/Backplane.kicad_pcb (KiCad board)
At the start: 2 copper layers, 100 x 100 mm, 14 parts, among them J1 Conn_02x20_Odd_Even, J2 Conn_02x20_Odd_Even, J3 Conn_02x20_Odd_Even, J4 Conn_02x20_Odd_Even, J5 Conn_02x20_Odd_Even, J6 6502 Bus, J7 6502 Bus

Commit message: Housekeeping
Parts:
- J1, J2, J3, J4, J5: value Conn_02x20_Odd_Even -> 6502 Card Connector
Changed lines of the file:
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@@
 		(sheetname "Root")
 		(sheetfile "Backplane.kicad_sch")
-		(attr exclude_from_pos_files exclude_from_bom)
+		(attr board_only exclude_from_pos_files exclude_from_bom)
 		(fp_circle
 			(center 0 0)
@@
 		(sheetname "Root")
 		(sheetfile "Backplane.kicad_sch")
-		(attr exclude_from_pos_files exclude_from_bom)
+		(attr board_only exclude_from_pos_files exclude_from_bom)
 		(fp_circle
 			(center 0 0)
@@
 			)
 		)
-		(property "Value" "Conn_02x20_Odd_Even"
+		(property "Value" "6502 Card Connector"
 			(at 0 0 90)
 			(layer "F.Fab")
@@
 			)
 		)
-		(property "Datasheet" ""
+		(property "Datasheet" "~"
 			(at 0 0 270)
 			(unlocked yes)
@@
 		)
 		(property ki_fp_filters "Connector*:*_2x??_*")
-		(sheetname "Root")
+		(sheetname "/")
 		(sheetfile "Backplane.kicad_sch")
 		(attr through_hole exclude_from_bom)
@@
 			)
 		)
-		(property "Value" "Conn_02x20_Odd_Even"
+		(property "Value" "6502 Card Connector"
 			(at 0 0 90)
 			(layer "F.Fab")
@@
 			)
 		)
-		(property "Datasheet" ""
+		(property "Datasheet" "~"
 			(at 0 0 270)
 			(unlocked yes)
@@
 		)
 		(property ki_fp_filters "Connector*:*_2x??_*")
-		(sheetname "Root")
+		(sheetname "/")
 		(sheetfile "Backplane.kicad_sch")
 		(attr through_hole exclude_from_bom)
@@
 			)
 		)
-		(property "Value" "Conn_02x20_Odd_Even"
+		(property "Value" "6502 Card Connector"
 			(at 0 0 90)
 			(layer "F.Fab")
@@
 			)
 		)
-		(property "Datasheet" ""
+		(property "Datasheet" "~"
 			(at 0 0 270)
 			(unlocked yes)
@@
 		)
 		(property ki_fp_filters "Connector*:*_2x??_*")
-		(sheetname "Root")
+		(sheetname "/")
 		(sheetfile "Backplane.kicad_sch")
 		(attr through_hole exclude_from_bom)
@@
 			)
 		)
-		(property "Value" "Conn_02x20_Odd_Even"
+		(property "Value" "6502 Card Connector"
 			(at 0 0 90)
 			(layer "F.Fab")
@@
 			)
 		)
-		(property "Datasheet" ""
+		(property "Datasheet" "~"
 			(at 0 0 270)
 			(unlocked yes)
@@
 		)
 		(property ki_fp_filters "Connector*:*_2x??_*")
-		(sheetname "Root")
+		(sheetname "/")
 		(sheetfile "Backplane.kicad_sch")
 		(attr through_hole exclude_from_bom)
@@
 		(sheetname "Root")
 		(sheetfile "Backplane.kicad_sch")
-		(attr exclude_from_pos_files exclude_from_bom)
+		(attr board_only exclude_from_pos_files exclude_from_bom)
 		(fp_circle
 			(center 0 0)
@@
 	)
 	(footprint "6502 Logos:6502 Backplane Logo 5mm"
-		(locked yes)
 		(layer "F.Cu")
 		(at 165.608 55.88 180)
@@
 			)
 		)
-		(attr through_hole)
+		(attr through_hole board_only exclude_from_pos_files exclude_from_bom allow_missing_courtyard)
 		(fp_poly
 			(pts
@@
 		(sheetname "Root")
 		(sheetfile "Backplane.kicad_sch")
-		(attr exclude_from_pos_files exclude_from_bom)
+		(attr board_only exclude_from_pos_files exclude_from_bom)
 		(fp_circle
 			(center 0 0)
@@
 			)
 		)
-		(property "Value" "Conn_02x20_Odd_Even"
+		(property "Value" "6502 Card Connector"
 			(at 0 0 90)
 			(layer "F.Fab")
@@
 			)
 		)
-		(property "Datasheet" ""
+		(property "Datasheet" "~"
 			(at 0 0 270)
 			(unlocked yes)
@@
 		)
 		(property ki_fp_filters "Connector*:*_2x??_*")
-		(sheetname "Root")
+		(sheetname "/")
 		(sheetfile "Backplane.kicad_sch")
 		(attr through_hole exclude_from_bom)
@@
 			)
 		)
-		(attr through_hole)
+		(attr through_hole board_only exclude_from_pos_files exclude_from_bom allow_missing_courtyard)
 		(fp_poly
 			(pts
@@
 			)
 		)
-		(attr exclude_from_pos_files exclude_from_bom allow_missing_courtyard)
+		(attr board_only exclude_from_pos_files exclude_from_bom allow_missing_courtyard)
 		(fp_poly
 			(pts
@@
 			)
 		)
-		(property "Datasheet" ""
+		(property "Datasheet" "~"
 			(at 0 0 0)
 			(unlocked yes)
@@
 			)
 		)
+		(property "Digikey" "732-5401-ND"
+			(at 0 0 0)
+			(unlocked yes)
+			(layer "F.Fab")
+			(hide yes)
+			(effects
+				(font
+					(size 1 1)
+					(thickness 0.15)
+				)
+			)
+		)
 		(property ki_fp_filters "Connector*:*_2x??_*")
-		(sheetname "Root")
+		(sheetname "/")
 		(sheetfile "Backplane.kicad_sch")
 		(attr through_hole exclude_from_bom)
@@
 			)
 		)
-		(property "Datasheet" ""
+		(property "Datasheet" "~"
 			(at 0 0 270)
 			(unlocked yes)
@@
 			)
 		)
+		(property "Digikey" "732-5401-ND"
+			(at 0 0 270)
+			(unlocked yes)
+			(layer "F.Fab")
+			(hide yes)
+			(effects
+				(font
+					(size 1 1)
+					(thickness 0.15)
+				)
+			)
+		)
 		(property ki_fp_filters "Connector*:*_2x??_*")
-		(sheetname "Root")
+		(sheetname "/")
 		(sheetfile "Backplane.kicad_sch")
 		(attr through_hole exclude_from_bom)
