File: Hardware/Backplane/Rev 1.0/Backplane.kicad_sch (KiCad schematic)
At the start: 11 parts, among them J1 Conn_02x20_Odd_Even, J2 Conn_02x20_Odd_Even, J3 Conn_02x20_Odd_Even, J4 Conn_02x20_Odd_Even, J5 Conn_02x20_Odd_Even, J6 6502 Bus, J7 6502 Bus

Commit message: Add 3D images for all boards
Parts:
- J6, J7: Digikey (none) -> 732-5401-ND
Changed lines of the file:
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@@
+			)
+		)
+		(property "Digikey" "732-5401-ND"
+			(at 60.96 137.16 0)
+			(effects
+				(font
+					(size 1.27 1.27)
+				)
+				(hide yes)
 			)
 		)
@@
 			(at 118.11 137.16 0)
 			(effects
+				(font
+					(size 1.27 1.27)
+				)
+				(hide yes)
+			)
+		)
+		(property "Digikey" "732-5401-ND"
+			(at 118.11 137.16 0)
+			(effects

Commit message: Edit schematics for clarity
Parts:
- J1, J2, J3, J4, J5: value Conn_02x20_Odd_Even -> 6502 Card Connector
Changed lines of the file:
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@@
 			)
 		)
-		(property "Value" "Conn_02x20_Odd_Even"
-			(at 60.96 26.0096 0)
-			(effects
-				(font
-					(size 1.27 1.27)
-				)
-				(hide yes)
+		(property "Value" "6502 Card Connector"
+			(at 61.214 81.026 0)
+			(effects
+				(font
+					(size 1.27 1.27)
+				)
 			)
 		)
@@
 			)
 		)
-		(property "Value" "Conn_02x20_Odd_Even"
-			(at 99.06 26.0096 0)
-			(effects
-				(font
-					(size 1.27 1.27)
-				)
-				(hide yes)
+		(property "Value" "6502 Card Connector"
+			(at 98.806 81.026 0)
+			(effects
+				(font
+					(size 1.27 1.27)
+				)
 			)
 		)
@@
 			)
 		)
-		(property "Value" "Conn_02x20_Odd_Even"
-			(at 137.16 26.0096 0)
-			(effects
-				(font
-					(size 1.27 1.27)
-				)
-				(hide yes)
+		(property "Value" "6502 Card Connector"
+			(at 137.16 81.026 0)
+			(effects
+				(font
+					(size 1.27 1.27)
+				)
 			)
 		)
@@
 			)
 		)
-		(property "Value" "Conn_02x20_Odd_Even"
-			(at 175.26 26.0096 0)
-			(effects
-				(font
-					(size 1.27 1.27)
-				)
-				(hide yes)
+		(property "Value" "6502 Card Connector"
+			(at 175.26 81.534 0)
+			(effects
+				(font
+					(size 1.27 1.27)
+				)
 			)
 		)
@@
 			)
 		)
-		(property "Value" "Conn_02x20_Odd_Even"
-			(at 213.36 26.0096 0)
-			(effects
-				(font
-					(size 1.27 1.27)
-				)
-				(hide yes)
-			)
-		)
+		(property "Value" "6502 Card Connector"
+			(at 213.36 81.534 0)
+			(effects
+				(font
+					(size 1.27 1.27)
+				)
+			)
+		)

Commit message: Housekeeping
Parts:
- removed H1, H2, H3, H4: MountingHole, MountingHole:MountingHole_3.2mm_M3, symbol Mechanical:MountingHole
