File: Hardware/Front Panel/Rev 1.0/Front Panel.kicad_pcb (KiCad board)
At the start: 2 copper layers, 100 x 100 mm, 18 parts, among them J1 PWR_SW, J2 RESET_SW, J3 CLOCK_ENBL_SW, J4 6502 Bus, J5 6502 Bus, SW1 Power, SW2 Reset, SW3 Run / Halt

Commit message: Replace switches on Front Panel board with SS12D10
Parts:
- SW1, SW2, SW3: footprint 6502 Parts:300SP1J1BLKM2QE -> 6502 Parts:SS12D10
Changed lines of the file:
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@@
 		)
 	)
-	(footprint "6502 Parts:300SP1J1BLKM2QE"
+	(footprint "6502 Parts:SS12D10"
 		(layer "F.Cu")
 		(at 140 100)
@@
 		)
 		(embedded_fonts no)
-		(model "${KIPRJMOD}/../../../CAD/300SP1J1BLKM2QE.step"
+		(model "${KIPRJMOD}/../../../CAD/SS12D10.step"
 			(offset
-				(xyz 0 0 0)
+				(xyz 0 0 0.5)
 			)
 			(scale
@@
 			)
 			(rotate
-				(xyz -90 0 0)
+				(xyz -0 -0 -90)
 			)
 		)
 	)
-	(footprint "6502 Parts:300SP1J1BLKM2QE"
+	(footprint "6502 Parts:SS12D10"
 		(layer "F.Cu")
 		(at 140 70)
@@
 		)
 		(embedded_fonts no)
-		(model "${KIPRJMOD}/../../../CAD/300SP1J1BLKM2QE.step"
+		(model "${KIPRJMOD}/../../../CAD/SS12D10.step"
 			(offset
-				(xyz 0 0 0)
+				(xyz 0 0 0.5)
 			)
 			(scale
@@
 			)
 			(rotate
-				(xyz -90 0 0)
+				(xyz -0 -0 -90)
 			)
 		)
 	)
-	(footprint "6502 Parts:300SP1J1BLKM2QE"
+	(footprint "6502 Parts:SS12D10"
 		(layer "F.Cu")
 		(at 140 85)
@@
 		)
 		(embedded_fonts no)
-		(model "${KIPRJMOD}/../../../CAD/300SP1J1BLKM2QE.step"
+		(model "${KIPRJMOD}/../../../CAD/SS12D10.step"
 			(offset
-				(xyz 0 0 0)
+				(xyz 0 0 0.5)
 			)
 			(scale
@@
 			)
 			(rotate
-				(xyz -90 0 0)
-			)
-		)
+				(xyz -0 -0 -90)
+			)
+		)
