File: Hardware/GPIO Breadboard Helper/Rev 1.0/GPIO Breadboard Helper.kicad_pcb (KiCad board)
At the start: 2 copper layers, 58.8 x 55 mm, 5 parts, among them J1 PORT A, J2 PORT A, J3 PORT B, J4 PORT B

Commit message: Housekeeping
Parts:
- added G***: LOGO, A.C. Wright Logo:A.C. Wright Logo 5mm, F.Cu at (135.4, 101.3)
- added REF**: OSHW-Logo2_7.3x6mm_SilkScreen, Symbol:OSHW-Logo2_7.3x6mm_SilkScreen, F.Cu at (97.0, 101.3)
