File: Hardware/Main Board/Rev 1.0/Main Board.kicad_pcb (KiCad board)
At the start: 2 copper layers, 100 x 100 mm, 63 parts, among them J1 PWR_SW, J10 Conn_02x20_Odd_Even, J2 Conn_02x01, J3 USB_C_Receptacle_USB2.0, J4 RESET_SW, J5 Conn_02x02_Odd_Even, J6 CLOCK_ENBL_SW, J7 Conn_01x02, J8 Conn_02x05_Odd_Even, J9 Conn_02x20_Odd_Even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

Commit message: Housekeeping
Parts:
- J10: value Conn_02x20_Odd_Even -> 6502 Bus
- J9: value Conn_02x20_Odd_Even -> 6502 Card Connector
