File: Hardware/Memory Card/Rev 1.0/Memory Card.kicad_pcb (KiCad board)
At the start: 2 copper layers, 100 x 57.6 mm, 26 parts, among them J1 6502 Card Edge, J2 Conn_02x02_Odd_Even, J3 Conn_02x01, U1 74HC00, U2 74HC00, U3 AS6C62256, U4 AT28C256, U5 74HC00

Commit message: Housekeeping
Connections:
- net /A0 renamed A0
- net /A1 renamed A1
- net /A10 renamed A10
- net /A11 renamed A11
- net /A12 renamed A12
- net /A2 renamed A2
- net /A3 renamed A3
- net /A4 renamed A4
- net /A5 renamed A5
- net /A6 renamed A6
- net /A7 renamed A7
- net /A8 renamed A8
- net /A9 renamed A9
- net /D0 renamed D0
- net /D1 renamed D1
- net /D2 renamed D2
- net /D3 renamed D3
- net /D4 renamed D4
- net /D5 renamed D5
- net /D6 renamed D6
- net /D7 renamed D7
