File: Hardware/Prototype Card/Rev 1.0/Prototype Card.kicad_pcb (KiCad board)
At the start: 2 copper layers, 100 x 57.6 mm, 12 parts, among them J1 6502 Card Edge, J2 Conn_02x20_Odd_Even, J3 Conn_02x04_Odd_Even, U1 74HC138

Commit message: Add 3D images for all boards
Parts:
- B1, B2: footprint 6502 Parts:BREADBOARD-MINI -> 6502 Parts:Breadboard Mini
Changed lines of the file:
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@@
 	(net 45 "/EXP2")
 	(net 46 "/EXP3")
-	(footprint "6502 Parts:BREADBOARD-MINI"
+	(footprint "6502 Parts:Breadboard Mini"
 		(layer "F.Cu")
 		(at 125.73 95.25)
@@
 		(property "Datasheet" ""
 			(at 0 0 0)
-			(unlocked yes)
 			(layer "F.Fab")
 			(hide yes)
@@
 		(property "Description" ""
 			(at 0 0 0)
-			(unlocked yes)
 			(layer "F.Fab")
 			(hide yes)
@@
 		)
 		(embedded_fonts no)
+		(model "${KIPRJMOD}/../../../CAD/Mini-Black.step"
+			(offset
+				(xyz 0 0 5)
+			)
+			(scale
+				(xyz 1 1 1)
+			)
+			(rotate
+				(xyz -90 -0 -0)
+			)
+		)
 	)
-	(footprint "6502 Parts:BREADBOARD-MINI"
+	(footprint "6502 Parts:Breadboard Mini"
 		(layer "F.Cu")
 		(at 171.45 95.25)
@@
 		(property "Datasheet" ""
 			(at 0 0 0)
-			(unlocked yes)
 			(layer "F.Fab")
 			(hide yes)
@@
 		(property "Description" ""
 			(at 0 0 0)
-			(unlocked yes)
 			(layer "F.Fab")
 			(hide yes)
@@
 		)
 		(embedded_fonts no)
+		(model "${KIPRJMOD}/../../../CAD/Mini-Black.step"
+			(offset
+				(xyz 0 0 5)
+			)
+			(scale
+				(xyz 1 1 1)
+			)
+			(rotate
+				(xyz -90 -0 -0)
+			)
+		)
 	)
 	(footprint "Capacitor_SMD:C_0805_2012Metric"

Commit message: Housekeeping
Connections:
- net /A0 renamed A0
- net /A1 renamed A1
- net /A2 renamed A2
- net /A3 renamed A3
- net /A4 renamed A4
- net /A5 renamed A5
- net /A6 renamed A6
- net /A7 renamed A7
- net /A8 renamed A8
- net /A9 renamed A9
- net /BE renamed BE
- net /D0 renamed D0
- net /D1 renamed D1
- net /D2 renamed D2
- net /D3 renamed D3
- net /D4 renamed D4
- net /D5 renamed D5
- net /D6 renamed D6
- net /D7 renamed D7
- net /EXP0 renamed EXP0
- net /EXP1 renamed EXP1
- net /EXP2 renamed EXP2
- net /EXP3 renamed EXP3
- net /IRQB renamed IRQB
- net /NMIB renamed NMIB
- net /PHI2 renamed PHI2
- net /RDY renamed RDY
- net /RESB renamed RESB
- net /RWB renamed RWB
- net /SYNC renamed SYNC
