File: Hardware/Keyboard Helper/Rev 1.0/Keyboard Helper.kicad_sch (KiCad schematic)
At the start: 87 parts, among them J1 PORT A, J2 PORT B, J3 KEYBOARD, J4 JOYSTICK A, J5 JOYSTICK B, J6 JOYSTICK A, J7 JOYSTICK B, SW1 DEL, SW10 R, SW11 D, SW12 6, SW13 7, SW14 Y, SW15 G, SW16 8, SW17 9, SW18 I, SW19 J, SW2 RETURN, SW20 0, SW21 +, SW22 P, SW23 L, SW24 -, SW25 £, SW26 *, SW27 ;, SW28 HOME, SW29 1, SW3 LEFT/RIGHT, SW30 LEFT ARROW, SW31 CTRL, SW32 2, SW33 F1, SW34 F3, SW35 F5, SW36 UP/DOWN, SW37 Z, SW38 S, SW39 E, SW4 F7, SW40 L SHIFT, SW41 C, SW42 F, SW43 T, SW44 X, SW45 B, SW46 H, SW47 U, SW48 V, SW49 M, SW5 3, SW50 K, SW51 O, SW52 N, SW53 ., SW54 :, SW55 @, SW56 ,, SW57 R SHIFT, SW58 =, SW59 UP ARROW, SW6 W, SW60 /, SW61 SPACE, SW62 C64, SW63 Q, SW64 RUN/STOP, SW7 A, SW8 4, SW9 5

Commit message: Progress on Keyboard Helper
Parts:
- added SW65: R SHIFT, 6502 Parts:SW_Cherry_MX_2.25u_PCB, symbol Switch:SW_Push
- added SW66: R ALT, 6502 Parts:SW_Cherry_MX_1.25u_PCB, symbol Switch:SW_Push
- added SW67: R CTRL, 6502 Parts:SW_Cherry_MX_1.25u_PCB, symbol Switch:SW_Push
- J1: renamed from J4; now left out of the parts list
- J2: renamed from J5; now left out of the parts list
- J7: renamed from J3; now left out of the parts list
- SW1: value DEL -> `; footprint Button_Switch_Keyboard:SW_Cherry_MX_1.00u_PCB -> 6502 Parts:SW_Cherry_MX_1.00u_PCB
- SW10: renamed from SW6; value W -> 9; footprint Button_Switch_Keyboard:SW_Cherry_MX_1.00u_PCB -> 6502 Parts:SW_Cherry_MX_1.00u_PCB
- SW11: renamed from SW7; value A -> 0; footprint Button_Switch_Keyboard:SW_Cherry_MX_1.00u_PCB -> 6502 Parts:SW_Cherry_MX_1.00u_PCB
- SW12: renamed from SW8; value 4 -> -; footprint Button_Switch_Keyboard:SW_Cherry_MX_1.00u_PCB -> 6502 Parts:SW_Cherry_MX_1.00u_PCB
- SW13: renamed from SW37; value Z -> =; footprint Button_Switch_Keyboard:SW_Cherry_MX_1.00u_PCB -> 6502 Parts:SW_Cherry_MX_1.00u_PCB
- SW14: renamed from SW38; value S -> BACKSPACE; footprint Button_Switch_Keyboard:SW_Cherry_MX_1.00u_PCB -> 6502 Parts:SW_Cherry_MX_2.00u_PCB
- SW15: renamed from SW39; value E -> ESCAPE; footprint Button_Switch_Keyboard:SW_Cherry_MX_1.00u_PCB -> 6502 Parts:SW_Cherry_MX_1.00u_PCB
- SW16: renamed from SW40; value L SHIFT -> TAB; footprint Button_Switch_Keyboard:SW_Cherry_MX_1.00u_PCB -> 6502 Parts:SW_Cherry_MX_1.50u_PCB
- SW17: renamed from SW9; value 5 -> Q; footprint Button_Switch_Keyboard:SW_Cherry_MX_1.00u_PCB -> 6502 Parts:SW_Cherry_MX_1.00u_PCB
- SW18: renamed from SW10; value R -> W; footprint Button_Switch_Keyboard:SW_Cherry_MX_1.00u_PCB -> 6502 Parts:SW_Cherry_MX_1.00u_PCB
- SW19: renamed from SW11; value D -> E; footprint Button_Switch_Keyboard:SW_Cherry_MX_1.00u_PCB -> 6502 Parts:SW_Cherry_MX_1.00u_PCB
- SW2: value RETURN -> 1; footprint Button_Switch_Keyboard:SW_Cherry_MX_1.00u_PCB -> 6502 Parts:SW_Cherry_MX_1.00u_PCB
- SW20: renamed from SW12; value 6 -> R; footprint Button_Switch_Keyboard:SW_Cherry_MX_1.00u_PCB -> 6502 Parts:SW_Cherry_MX_1.00u_PCB
- SW21: renamed from SW41; value C -> T; footprint Button_Switch_Keyboard:SW_Cherry_MX_1.00u_PCB -> 6502 Parts:SW_Cherry_MX_1.00u_PCB
- SW22: renamed from SW42; value F -> Y; footprint Button_Switch_Keyboard:SW_Cherry_MX_1.00u_PCB -> 6502 Parts:SW_Cherry_MX_1.00u_PCB
- SW23: renamed from SW43; value T -> U; footprint Button_Switch_Keyboard:SW_Cherry_MX_1.00u_PCB -> 6502 Parts:SW_Cherry_MX_1.00u_PCB
- SW24: renamed from SW44; value X -> I; footprint Button_Switch_Keyboard:SW_Cherry_MX_1.00u_PCB -> 6502 Parts:SW_Cherry_MX_1.00u_PCB
- SW25: renamed from SW13; value 7 -> O; footprint Button_Switch_Keyboard:SW_Cherry_MX_1.00u_PCB -> 6502 Parts:SW_Cherry_MX_1.00u_PCB
- SW26: renamed from SW14; value Y -> P; footprint Button_Switch_Keyboard:SW_Cherry_MX_1.00u_PCB -> 6502 Parts:SW_Cherry_MX_1.00u_PCB
- SW27: renamed from SW15; value G -> [; footprint Button_Switch_Keyboard:SW_Cherry_MX_1.00u_PCB -> 6502 Parts:SW_Cherry_MX_1.00u_PCB
- SW28: renamed from SW16; value 8 -> ]; footprint Button_Switch_Keyboard:SW_Cherry_MX_1.00u_PCB -> 6502 Parts:SW_Cherry_MX_1.00u_PCB
- SW29: renamed from SW45; value B -> \; footprint Button_Switch_Keyboard:SW_Cherry_MX_1.00u_PCB -> 6502 Parts:SW_Cherry_MX_1.50u_PCB
- SW3: value LEFT/RIGHT -> 2; footprint Button_Switch_Keyboard:SW_Cherry_MX_1.00u_PCB -> 6502 Parts:SW_Cherry_MX_1.00u_PCB
- SW30: renamed from SW46; value H -> INSERT; footprint Button_Switch_Keyboard:SW_Cherry_MX_1.00u_PCB -> 6502 Parts:SW_Cherry_MX_1.00u_PCB
- SW31: renamed from SW47; value U -> CAPS LOCK; footprint Button_Switch_Keyboard:SW_Cherry_MX_1.00u_PCB -> 6502 Parts:SW_Cherry_MX_1.75u_PCB
- SW32: renamed from SW48; value V -> A; footprint Button_Switch_Keyboard:SW_Cherry_MX_1.00u_PCB -> 6502 Parts:SW_Cherry_MX_1.00u_PCB
- SW33: renamed from SW17; value 9 -> S; footprint Button_Switch_Keyboard:SW_Cherry_MX_1.00u_PCB -> 6502 Parts:SW_Cherry_MX_1.00u_PCB
- SW34: renamed from SW18; value I -> D; footprint Button_Switch_Keyboard:SW_Cherry_MX_1.00u_PCB -> 6502 Parts:SW_Cherry_MX_1.00u_PCB
- SW35: renamed from SW19; value J -> F; footprint Button_Switch_Keyboard:SW_Cherry_MX_1.00u_PCB -> 6502 Parts:SW_Cherry_MX_1.00u_PCB
- SW36: renamed from SW20; value 0 -> G; footprint Button_Switch_Keyboard:SW_Cherry_MX_1.00u_PCB -> 6502 Parts:SW_Cherry_MX_1.00u_PCB
- SW37: renamed from SW49; value M -> H; footprint Button_Switch_Keyboard:SW_Cherry_MX_1.00u_PCB -> 6502 Parts:SW_Cherry_MX_1.00u_PCB
- SW38: renamed from SW50; value K -> J; footprint Button_Switch_Keyboard:SW_Cherry_MX_1.00u_PCB -> 6502 Parts:SW_Cherry_MX_1.00u_PCB
- SW39: renamed from SW51; value O -> K; footprint Button_Switch_Keyboard:SW_Cherry_MX_1.00u_PCB -> 6502 Parts:SW_Cherry_MX_1.00u_PCB
- SW4: value F7 -> 3; footprint Button_Switch_Keyboard:SW_Cherry_MX_1.00u_PCB -> 6502 Parts:SW_Cherry_MX_1.00u_PCB
- SW40: renamed from SW52; value N -> L; footprint Button_Switch_Keyboard:SW_Cherry_MX_1.00u_PCB -> 6502 Parts:SW_Cherry_MX_1.00u_PCB
- SW41: renamed from SW21; value + -> ;; footprint Button_Switch_Keyboard:SW_Cherry_MX_1.00u_PCB -> 6502 Parts:SW_Cherry_MX_1.00u_PCB
- SW42: renamed from SW22; value P -> '; footprint Button_Switch_Keyboard:SW_Cherry_MX_1.00u_PCB -> 6502 Parts:SW_Cherry_MX_1.00u_PCB
- SW43: renamed from SW23; value L -> ENTER; footprint Button_Switch_Keyboard:SW_Cherry_MX_1.00u_PCB -> 6502 Parts:SW_Cherry_MX_2.25u_PCB
- SW44: renamed from SW24; value - -> DELETE; footprint Button_Switch_Keyboard:SW_Cherry_MX_1.00u_PCB -> 6502 Parts:SW_Cherry_MX_1.00u_PCB
- SW45: renamed from SW53; value . -> SHIFT; footprint Button_Switch_Keyboard:SW_Cherry_MX_1.00u_PCB -> 6502 Parts:SW_Cherry_MX_2.25u_PCB
- SW46: renamed from SW54; value : -> Z; footprint Button_Switch_Keyboard:SW_Cherry_MX_1.00u_PCB -> 6502 Parts:SW_Cherry_MX_1.00u_PCB
- SW47: renamed from SW55; value @ -> X; footprint Button_Switch_Keyboard:SW_Cherry_MX_1.00u_PCB -> 6502 Parts:SW_Cherry_MX_1.00u_PCB
- SW48: renamed from SW56; value , -> C; footprint Button_Switch_Keyboard:SW_Cherry_MX_1.00u_PCB -> 6502 Parts:SW_Cherry_MX_1.00u_PCB
- SW49: renamed from SW25; value £ -> V; footprint Button_Switch_Keyboard:SW_Cherry_MX_1.00u_PCB -> 6502 Parts:SW_Cherry_MX_1.00u_PCB
- SW5: renamed from SW33; value F1 -> 4; footprint Button_Switch_Keyboard:SW_Cherry_MX_1.00u_PCB -> 6502 Parts:SW_Cherry_MX_1.00u_PCB
- SW50: renamed from SW26; value * -> B; footprint Button_Switch_Keyboard:SW_Cherry_MX_1.00u_PCB -> 6502 Parts:SW_Cherry_MX_1.00u_PCB
- SW51: renamed from SW27; value ; -> N; footprint Button_Switch_Keyboard:SW_Cherry_MX_1.00u_PCB -> 6502 Parts:SW_Cherry_MX_1.00u_PCB
- SW52: renamed from SW28; value HOME -> M; footprint Button_Switch_Keyboard:SW_Cherry_MX_1.00u_PCB -> 6502 Parts:SW_Cherry_MX_1.00u_PCB
- SW53: renamed from SW57; value R SHIFT -> ,; footprint Button_Switch_Keyboard:SW_Cherry_MX_1.00u_PCB -> 6502 Parts:SW_Cherry_MX_1.00u_PCB
- SW54: renamed from SW58; value = -> .; footprint Button_Switch_Keyboard:SW_Cherry_MX_1.00u_PCB -> 6502 Parts:SW_Cherry_MX_1.00u_PCB
- SW55: renamed from SW59; value UP ARROW -> /; footprint Button_Switch_Keyboard:SW_Cherry_MX_1.00u_PCB -> 6502 Parts:SW_Cherry_MX_1.00u_PCB
- SW56: renamed from SW60; value / -> UP ARROW; footprint Button_Switch_Keyboard:SW_Cherry_MX_1.00u_PCB -> 6502 Parts:SW_Cherry_MX_1.00u_PCB
- SW57: renamed from SW29; value 1 -> CTRL; footprint Button_Switch_Keyboard:SW_Cherry_MX_1.00u_PCB -> 6502 Parts:SW_Cherry_MX_1.25u_PCB
- SW58: renamed from SW30; value LEFT ARROW -> MENU; footprint Button_Switch_Keyboard:SW_Cherry_MX_1.00u_PCB -> 6502 Parts:SW_Cherry_MX_1.00u_PCB
- SW59: renamed from SW31; value CTRL -> ALT; footprint Button_Switch_Keyboard:SW_Cherry_MX_1.00u_PCB -> 6502 Parts:SW_Cherry_MX_1.25u_PCB
- SW6: renamed from SW34; value F3 -> 5; footprint Button_Switch_Keyboard:SW_Cherry_MX_1.00u_PCB -> 6502 Parts:SW_Cherry_MX_1.00u_PCB
- SW60: renamed from SW32; value 2 -> SPACE; footprint Button_Switch_Keyboard:SW_Cherry_MX_1.00u_PCB -> 6502 Parts:SW_Cherry_MX_6.25u_PCB
- SW61: value SPACE -> FN; footprint Button_Switch_Keyboard:SW_Cherry_MX_1.00u_PCB -> 6502 Parts:SW_Cherry_MX_1.25u_PCB
- SW62: value C64 -> LEFT ARROW; footprint Button_Switch_Keyboard:SW_Cherry_MX_1.00u_PCB -> 6502 Parts:SW_Cherry_MX_1.00u_PCB
- SW63: value Q -> DOWN ARROW; footprint Button_Switch_Keyboard:SW_Cherry_MX_1.00u_PCB -> 6502 Parts:SW_Cherry_MX_1.00u_PCB
- SW64: value RUN/STOP -> RIGHT ARROW; footprint Button_Switch_Keyboard:SW_Cherry_MX_1.00u_PCB -> 6502 Parts:SW_Cherry_MX_1.00u_PCB
- SW7: renamed from SW35; value F5 -> 6; footprint Button_Switch_Keyboard:SW_Cherry_MX_1.00u_PCB -> 6502 Parts:SW_Cherry_MX_1.00u_PCB
- SW8: renamed from SW36; value UP/DOWN -> 7; footprint Button_Switch_Keyboard:SW_Cherry_MX_1.00u_PCB -> 6502 Parts:SW_Cherry_MX_1.00u_PCB
- SW9: renamed from SW5; value 3 -> 8; footprint Button_Switch_Keyboard:SW_Cherry_MX_1.00u_PCB -> 6502 Parts:SW_Cherry_MX_1.00u_PCB
- renumbered J6 to J3, J7 to J4, J1 to J5, J2 to J6
Connections:
- net PA5: now also SW65.1
- net PA7: now also SW66.1, SW67.1
- net PB0: now also SW67.2
- net PB2: now also SW66.2
- net PB4: now also SW65.2
Other:
- moved on the sheet: SW45, SW57, SW59
