File: Hardware/RTC Card/Rev 1.0/RTC Card.kicad_pcb (KiCad board)
At the start: 2 copper layers, 100 x 57.6 mm, 19 parts, among them J1 6502 Card Edge, J2 AUX, J3 INT Select, J4 Conn_02x08_Odd_Even, U1 DS1511Y, U2 74HC138, U3 74HC138

Commit message: Production fixes
Other:
- board text added: "JLCJLCJLCJLC"
Changed lines of the file:
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@@
+		)
+	)
+	(gr_text "JLCJLCJLCJLC"
+		(at 136.39 88.98 0)
+		(layer "F.SilkS")
+		(effects
+			(font
+				(size 1 1)
+				(thickness 0.15)
+			)
 		)
 	)
