File: Hardware/Nano Card/Rev 1.0/Nano Card.kicad_pcb (KiCad board)
At the start: 2 copper layers, 100 x 57.6 mm, 11 parts, among them J1 6502 Card Edge, U1 74HC595, U2 74HC595, U3 74HC595

Commit message: Cleanup for production
Connections:
- A1 pad 16: unconnected-(A1-D13-Pad16) -> DDATA
- A1 pad 7: unconnected-(A1-D4-Pad7) -> ADATA
- U1 pad 14: unconnected-(U1-SER-Pad14) -> ADATA
- U2 pad 14: unconnected-(U2-SER-Pad14) -> DDATA
Routing:
- net DDATA: track 0.00 -> 65.3 mm, vias 0 -> 4
- net ADATA: track 0.00 -> 49.6 mm, vias 0 -> 2
- net GND: vias 18 -> 17
Changed lines of the file:
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@@
 	(net 10 "unconnected-(J1-PadEXP2)")
 	(net 11 "DOEB")
-	(net 12 "unconnected-(A1-D4-Pad7)")
+	(net 12 "ADATA")
 	(net 13 "unconnected-(A1-3V3-Pad17)")
 	(net 14 "unconnected-(A1-~{RESET}-Pad3)")
@@
 	(net 32 "D2")
 	(net 33 "A13")
-	(net 34 "unconnected-(A1-D13-Pad16)")
+	(net 34 "DDATA")
 	(net 35 "D3")
 	(net 36 "unconnected-(A1-VIN-Pad30)")
@@
 	(net 49 "A8")
 	(net 50 "A6")
-	(net 51 "unconnected-(U1-SER-Pad14)")
-	(net 52 "Net-(U1-QH')")
-	(net 53 "unconnected-(U2-SER-Pad14)")
-	(net 54 "unconnected-(U2-QH&apos;-Pad9)")
-	(net 55 "unconnected-(U3-QH&apos;-Pad9)")
+	(net 51 "Net-(U1-QH')")
+	(net 52 "unconnected-(U2-QH&apos;-Pad9)")
+	(net 53 "unconnected-(U3-QH&apos;-Pad9)")
 	(footprint "Package_SO:SOIC-16_3.9x9.9mm_P1.27mm"
 		(layer "F.Cu")
@@
 			(layers "F.Cu" "F.Mask" "F.Paste")
 			(roundrect_rratio 0.25)
-			(net 55 "unconnected-(U3-QH&apos;-Pad9)")
+			(net 53 "unconnected-(U3-QH&apos;-Pad9)")
 			(pinfunction "QH'")
 			(pintype "output+no_connect")
@@
 			(layers "F.Cu" "F.Mask" "F.Paste")
 			(roundrect_rratio 0.25)
-			(net 52 "Net-(U1-QH')")
+			(net 51 "Net-(U1-QH')")
 			(pinfunction "SER")
 			(pintype "input")
@@
 			(layers "F.Cu" "F.Mask" "F.Paste")
 			(roundrect_rratio 0.25)
-			(net 52 "Net-(U1-QH')")
+			(net 51 "Net-(U1-QH')")
 			(pinfunction "QH'")
 			(pintype "output")
@@
 			(layers "F.Cu" "F.Mask" "F.Paste")
 			(roundrect_rratio 0.25)
-			(net 51 "unconnected-(U1-SER-Pad14)")
+			(net 12 "ADATA")
 			(pinfunction "SER")
 			(pintype "input")
@@
 			(layers "*.Cu" "*.Mask")
 			(remove_unused_layers no)
-			(net 12 "unconnected-(A1-D4-Pad7)")
+			(net 12 "ADATA")
 			(pinfunction "D4")
-			(pintype "bidirectional+no_connect")
+			(pintype "bidirectional")
 		)
 		(pad "8" thru_hole oval
@@
 			(layers "*.Cu" "*.Mask")
 			(remove_unused_layers no)
-			(net 34 "unconnected-(A1-D13-Pad16)")
+			(net 34 "DDATA")
 			(pinfunction "D13")
-			(pintype "bidirectional+no_connect")
+			(pintype "bidirectional")
 		)
 		(pad "17" thru_hole oval
@@
 			(layers "F.Cu" "F.Mask" "F.Paste")
 			(roundrect_rratio 0.25)
-			(net 54 "unconnected-(U2-QH&apos;-Pad9)")
+			(net 52 "unconnected-(U2-QH&apos;-Pad9)")
 			(pinfunction "QH'")
 			(pintype "output+no_connect")
@@
 			(layers "F.Cu" "F.Mask" "F.Paste")
 			(roundrect_rratio 0.25)
-			(net 53 "unconnected-(U2-SER-Pad14)")
+			(net 34 "DDATA")
 			(pinfunction "SER")
 			(pintype "input")
@@
 	)
 	(via
-		(at 158.54 103.95)
-		(size 0.6)
-		(drill 0.3)
-		(layers "F.Cu" "B.Cu")
-		(free yes)
-		(net 2)
-	)
-	(via
 		(at 149.32 112.77)
 		(size 0.6)
@@
 	)
 	(segment
+		(start 166.17 102.53)
+		(end 166.17 104.48)
+		(width 0.2)
+		(layer "F.Cu")
+		(net 12)
+	)
+	(segment
+		(start 125.16 99.42)
+		(end 124.96 99.22)
+		(width 0.2)
+		(layer "F.Cu")
+		(net 12)
+	)
+	(segment
+		(start 124.96 99.22)
+		(end 124.96 97.39)
+		(width 0.2)
+		(layer "F.Cu")
+		(net 12)
+	)
+	(segment
+		(start 125.16 103.56)
+		(end 125.16 99.42)
+		(width 0.2)
+		(layer "F.Cu")
+		(net 12)
+	)
+	(via
+		(at 166.17 104.48)
+		(size 0.6)
+		(drill 0.3)
+		(layers "F.Cu" "B.Cu")
+		(net 12)
+	)
+	(via
+		(at 125.16 103.56)
+		(size 0.6)
+		(drill 0.3)
+		(layers "F.Cu" "B.Cu")
+		(net 12)
+	)
+	(segment
+		(start 166.17 104.48)
+		(end 166.029 104.339)
+		(width 0.2)
+		(layer "B.Cu")
+		(net 12)
+	)
+	(segment
+		(start 166.029 104.339)
+		(end 125.939 104.339)
+		(width 0.2)
+		(layer "B.Cu")
+		(net 12)
+	)
+	(segment
+		(start 125.939 104.339)
+		(end 125.16 103.56)
+		(width 0.2)
+		(layer "B.Cu")
+		(net 12)
+	)
+	(segment
 		(start 108.43 97.36)
 		(end 107.16 97.36)
@@
 	)
 	(segment
+		(start 149.43 90.27)
+		(end 149.43 101.05)
+		(width 0.2)
+		(layer "F.Cu")
+		(net 34)
+	)
+	(segment
+		(start 186.49 90.09)
+		(end 186.49 87.29)
+		(width 0.2)
+		(layer "F.Cu")
+		(net 34)
+	)
+	(segment
+		(start 138.66 97.39)
+		(end 138.66 101.01)
+		(width 0.2)
+		(layer "F.Cu")
+		(net 34)
+	)
+	(segment
+		(start 149.41 90.25)
+		(end 149.43 90.27)
+		(width 0.2)
+		(layer "F.Cu")
+		(net 34)
+	)
+	(segment
+		(start 138.66 101.01)
+		(end 138.62 101.05)
+		(width 0.2)
+		(layer "F.Cu")
+		(net 34)
+	)
+	(segment
+		(start 149.41 90.1)
+		(end 149.41 90.25)
+		(width 0.2)
+		(layer "F.Cu")
+		(net 34)
+	)
+	(via
+		(at 149.43 101.05)
+		(size 0.6)
+		(drill 0.3)
+		(layers "F.Cu" "B.Cu")
+		(net 34)
+	)
+	(via
+		(at 186.49 90.09)
+		(size 0.6)
+		(drill 0.3)
+		(layers "F.Cu" "B.Cu")
+		(net 34)
+	)
+	(via
+		(at 149.41 90.1)
+		(size 0.6)
+		(drill 0.3)
+		(layers "F.Cu" "B.Cu")
+		(net 34)
+	)
+	(via
+		(at 138.62 101.05)
+		(size 0.6)
+		(drill 0.3)
+		(layers "F.Cu" "B.Cu")
+		(net 34)
+	)
+	(segment
+		(start 149.43 90.12)
+		(end 186.46 90.12)
+		(width 0.2)
+		(layer "B.Cu")
+		(net 34)
+	)
+	(segment
+		(start 186.46 90.12)
+		(end 186.49 90.09)
+		(width 0.2)
+		(layer "B.Cu")
+		(net 34)
+	)
+	(segment
+		(start 149.43 101.05)
+		(end 138.62 101.05)
+		(width 0.2)
+		(layer "B.Cu")
+		(net 34)
+	)
+	(segment
+		(start 149.41 90.1)
+		(end 149.43 90.12)
+		(width 0.2)
+		(layer "B.Cu")
+		(net 34)
+	)
+	(segment
 		(start 171.25 80.78)
 		(end 171.25 87.29)
@@
 		(width 0.2)
 		(layer "F.Cu")
-		(net 52)
+		(net 51)
 	)
 	(segment
@@
 		(width 0.2)
 		(layer "F.Cu")
-		(net 52)
+		(net 51)
 	)
 	(segment
@@
 		(width 0.2)
 		(layer "F.Cu")
-		(net 52)
+		(net 51)
 	)
 	(segment
@@
 		(width 0.2)
 		(layer "F.Cu")
-		(net 52)
+		(net 51)
 	)
 	(via
@@
 		(drill 0.3)
 		(layers "F.Cu" "B.Cu")
-		(net 52)
+		(net 51)
 	)
 	(via
@@
 		(drill 0.3)
 		(layers "F.Cu" "B.Cu")
-		(net 52)
+		(net 51)
 	)
 	(segment
@@
 		(width 0.2)
 		(layer "B.Cu")
-		(net 52)
+		(net 51)
 	)
 	(segment
@@
 		(width 0.2)
 		(layer "B.Cu")
-		(net 52)
+		(net 51)
 	)
 	(zone

Commit message: Production fixes
Other:
- board text added: "JLCJLCJLCJLC"
Changed lines of the file:
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@@
 		)
 		(property "Value" "Arduino Nano"
-			(at 8.89 19.05 180)
-			(layer "F.Fab")
+			(at 9.96 18.98 180)
+			(layer "F.SilkS")
 			(effects
 				(font
@@
 		(layer "Edge.Cuts")
 	)
+	(gr_text "JLCJLCJLCJLC"
+		(at 169.98 94.92 0)
+		(layer "F.SilkS")
+		(effects
+			(font
+				(size 1 1)
+				(thickness 0.15)
+			)
+		)
+	)
 	(gr_text "© 2024 A.C. Wright Design | acwrightdesign.com | Rev 1.0"
