File: Hardware/Dev Board/Rev 1.0/Dev Board.kicad_sch (KiCad schematic)
At the start: 40 parts, among them J1 VBAT, J2 SPI, J3 PANEL, J4 6502 Card Connector, J5 6502 Bus, J6 USB Host, J7 USB HOST, J8 RJ45_LED, J9 ETHERNET, SW1 Run/Stop, SW2 Step, SW3 Clock, SW4 Reset, U1 SN74LVC4245APWR, U2 SN74LVC4245APWR, U3 SN74LVC4245APWR, U4 Teensy4.1, U5 SN74LVC4245APWR, U6 SN74LVC4245APWR

Commit message: Changes to Dev Board
Parts:
- removed JP1: SolderJumper_2_Bridged, Jumper:SolderJumper-2_P1.3mm_Bridged_RoundedPad1.0x1.5mm, symbol Jumper:SolderJumper_2_Bridged
- removed R5: 1k, Resistor_SMD:R_0805_2012Metric, symbol Device:R
- added R11: 150, Resistor_SMD:R_0805_2012Metric, symbol Device:R
- renumbered R11 to R10, R6 to R5, R7 to R6, R8 to R7, R9 to R8, R10 to R9
Connections:
- net 3V3: now also R11.2
- net EXP0: no longer U6.7 (A5)
- net GND: now also J8.11, U6.7 (A5); no longer J2.7 (Pin_7)
- net at J8.12: now also R11.1
- net EXP0_3V3: no longer names the net of U6.17 (B5)
- net EXP0_3V3: no longer U4.31 (39_MISO1_OUT1A)
- net VBAT: no longer names the net of BT1.+, J1.1 (Pin_1), U4.50 (VBAT)
- new net CS2: J2.7 (Pin_7), U4.31 (39_MISO1_OUT1A)
- no-connect marks 18 -> 17
Other:
- moved on the sheet: J1

Commit message: Production fixes
Parts:
- BT1, J2, J3, U4: now left out of the parts list
Changed lines of the file:
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@@
 		(unit 1)
 		(exclude_from_sim no)
-		(in_bom yes)
+		(in_bom no)
 		(on_board yes)
 		(dnp no)
@@
 		(unit 1)
 		(exclude_from_sim no)
-		(in_bom yes)
+		(in_bom no)
 		(on_board yes)
 		(dnp no)
@@
 		(unit 1)
 		(exclude_from_sim no)
-		(in_bom yes)
+		(in_bom no)
 		(on_board yes)
 		(dnp no)
@@
 		(unit 1)
 		(exclude_from_sim no)
-		(in_bom yes)
+		(in_bom no)
 		(on_board yes)
 		(dnp no)
