File: Hardware/RAM Card/Rev 1.0/RAM Card.kicad_sch (KiCad schematic)
At the start: 18 parts, among them J1 6502 Card Edge, J2 Conn_02x08_Odd_Even, U1 AS6C4008, U2 74HC573, U3 74HC00, U4 74HC21, U5 74HC30, U6 74HC00, U7 74HC138

Commit message: RAM Card PCB
Parts:
- added J2: LATCH EN, Connector_PinHeader_2.54mm:PinHeader_1x02_P2.54mm_Vertical, symbol Connector_Generic:Conn_02x01
- added J4: BANK ADDR, Connector_PinHeader_2.54mm:PinHeader_2x05_P2.54mm_Vertical, symbol Connector_Generic:Conn_02x05_Odd_Even
- added JP1: Latch Enable, Jumper:SolderJumper-2_P1.3mm_Bridged_RoundedPad1.0x1.5mm, symbol Jumper:SolderJumper_2_Bridged
- renumbered C7 to C1, C1 to C2, C2 to C3, C3 to C4, C4 to C5, C5 to C6, C6 to C7, J2 to J3
Connections:
- net B10: now also J4.1 (Pin_1)
- net B11: now also J4.2 (Pin_2)
- net B12: now also J4.3 (Pin_3)
- net B13: now also J4.4 (Pin_4)
- net B14: now also J4.5 (Pin_5)
- net B15: now also J4.6 (Pin_6)
- net B16: now also J4.7 (Pin_7)
- net B17: now also J4.8 (Pin_8)
- net GND: now also J2.1 (Pin_1), J4.10 (Pin_10), JP1.1 (A); no longer U2.1 (OE)
- net VCC: now also J4.9 (Pin_9)
- new net: J2.2 (Pin_2), JP1.2 (B), U2.1 (OE)

Commit message: Production fixes
Parts:
- U1: now left out of the parts list
Changed lines of the file:
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@@
 		(unit 1)
 		(exclude_from_sim no)
-		(in_bom yes)
+		(in_bom no)
 		(on_board yes)
 		(dnp no)
