File: Hardware/DB25 Helper/Rev 1.0/DB25 Helper.kicad_sch (KiCad schematic)
At the start: 3 parts, among them J1 PORT A, J2 PORT B, J3 KEYBOARD

Commit message: Rename DB25 Helper
Other:
- title: 6502 GPIO DB25 Helper -> 6502 DB25 Helper
Changed lines of the file:
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@@
 	(paper "USLetter")
 	(title_block
-		(title "6502 GPIO DB25 Helper")
+		(title "6502 DB25 Helper")
 		(date "2025-09-28")
 		(rev "1.0")
