File: Hardware/Video Card Pro/Rev 1.0/Video Card Pro.kicad_sch (KiCad schematic)
At the start: 34 parts, among them J1 VIDEO, J2 SERIAL, J3 INT Select, J4 6502 Card Edge, J5 Conn_02x08_Odd_Even, Q1 2N4401, U1 74HC157, U2 74HC166, U3 ATmega1284-P, U4 74HC157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

Commit message: Video Card Pro schematic fix
Parts:
- Y1: value 16 MHz -> 14.31818 MHz
Changed lines of the file:
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@@
 			)
 		)
-		(property "Value" "16 MHz"
+		(property "Value" "14.31818 MHz"
 			(at 75.438 49.784 90)
 			(effects

Commit message: Video Card Pro PCB
Parts:
- removed C11: 100nF, Capacitor_SMD:C_0805_2012Metric, symbol Device:C
Changed lines of the file:
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@@
 	)
 	(junction
-		(at 311.15 125.73)
-		(diameter 0)
-		(color 0 0 0 0)
-	)
-	(junction
 		(at 143.51 165.1)
 		(diameter 0)
@@
 	)
 	(junction
-		(at 311.15 153.67)
-		(diameter 0)
-		(color 0 0 0 0)
-	)
-	(junction
 		(at 307.34 49.53)
 		(diameter 0)
@@
 	(wire
 		(pts
-			(xy 322.58 143.51) (xy 322.58 153.67)
-		)
-		(stroke
-			(width 0)
-			(type default)
-		)
-	)
-	(wire
-		(pts
 			(xy 119.38 101.6) (xy 123.19 101.6)
 		)
@@
 	(wire
 		(pts
-			(xy 322.58 125.73) (xy 311.15 125.73)
-		)
-		(stroke
-			(width 0)
-			(type default)
-		)
-	)
-	(wire
-		(pts
 			(xy 143.51 160.02) (xy 140.97 160.02)
 		)
@@
 	(wire
 		(pts
-			(xy 322.58 135.89) (xy 322.58 125.73)
-		)
-		(stroke
-			(width 0)
-			(type default)
-		)
-	)
-	(wire
-		(pts
 			(xy 265.43 125.73) (xy 254 125.73)
 		)
@@
 	(wire
 		(pts
-			(xy 322.58 153.67) (xy 311.15 153.67)
-		)
-		(stroke
-			(width 0)
-			(type default)
-		)
-	)
-	(wire
-		(pts
 			(xy 119.38 78.74) (xy 123.19 78.74)
 		)
@@
 					(unit 1)
 				)
-			)
-		)
-	)
-	(symbol
-		(lib_id "Device:C")
-		(at 322.58 139.7 0)
-		(unit 1)
-		(exclude_from_sim no)
-		(in_bom yes)
-		(on_board yes)
-		(dnp no)
-		(property "Reference" "C11"
-			(at 328.9808 139.7 90)
-			(effects
-				(font
-					(size 1.27 1.27)
-				)
-			)
-		)
-		(property "Value" "100nF"
-			(at 326.6694 139.7 90)
-			(effects
-				(font
-					(size 1.27 1.27)
-				)
-			)
-		)
-		(property "Footprint" "Capacitor_SMD:C_0805_2012Metric"
-			(at 323.5452 143.51 0)
-			(effects
-				(font
-					(size 1.27 1.27)
-				)
-				(hide yes)
-			)
-		)
-		(property "Datasheet" "~"
-			(at 322.58 139.7 0)
-			(effects
-				(font
-					(size 1.27 1.27)
-				)
-				(hide yes)
-			)
-		)
-		(property "Description" ""
-			(at 322.58 139.7 0)
-			(effects
-				(font
-					(size 1.27 1.27)
-				)
-				(hide yes)
-			)
-		)
-		(property "LCSC" "C49678"
-			(at 322.58 139.7 0)
-			(effects
-				(font
-					(size 1.27 1.27)
-				)
-				(hide yes)
-			)
-		)
-		(pin "1"
-		)
-		(pin "2"
-		)
-		(instances
-			(project "Video Card"
-				(path "/154a5133-b84f-49cb-b657-9c810539146c"
-					(reference "C11")
-					(unit 1)
-				)
