File: Hardware/Storage Card Pro/Rev 1.0/Storage Card Pro.kicad_sch (KiCad schematic)
At the start: 26 parts, among them J1 ACT LED, J2 6502 Card Edge, J3 SPI, J4 SD CARD, J5 Conn_02x08_Odd_Even, U1 TXS0108EPW, U2 ATmega328, U3 W25Q128JVS, U4 74HC138, U5 LP2985-3.3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

Commit message: Production fixes
Parts:
- U5: LCSC C47411546 -> C95414
Changed lines of the file:
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@@
 			)
 		)
-		(property "LCSC" "C47411546"
+		(property "LCSC" "C95414"
 			(at 129.54 177.8 0)
 			(effects
