File: Hardware/CPU Card Pro/Rev 1.0/CPU Card Pro.kicad_pcb (KiCad board)
At the start: 2 copper layers, 100 x 57.6 mm, 21 parts, among them J1 6502 Card Edge, J2 BANK ADDR, J3 EXP, U1 65C816, U2 74HC00, U3 74HC245, U4 74HC573, X1 OCXO-14

Commit message: RAM Card PCB
Changed lines of the file:
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@@
 			(effects
 				(font
-					(size 1 1)
+					(size 0.8 0.8)
 					(thickness 0.15)
 				)
@@
 	)
 	(gr_circle
+		(center 178.8011 86.1636)
+		(end 179.0011 86.1636)
+		(stroke
+			(width 0.4)
+			(type solid)
+		)
+		(fill no)
+		(layer "F.SilkS")
+	)
+	(gr_circle

Commit message: Remove oscillator from CPU cards
Parts:
- removed X1: OCXO-14, Oscillator:Oscillator_DIP-14
Routing:
- net PHI2: track 134.8 -> 85.1 mm, vias 6 -> 4
- net VCC: track 239.5 -> 233.3 mm, vias 14 -> 13
