File: Hardware/CPU Card/Rev 1.0/CPU Card.kicad_pcb (KiCad board)
At the start: 2 copper layers, 100 x 57.6 mm, 16 parts, among them J1 6502 Card Edge, J2 Conn_01x02, J3 Conn_02x05_Odd_Even, U1 65C02, X1 OCXO-14

Commit message: CPU Card minor silkscreen fix
Parts:
- J3: value Conn_02x05_Odd_Even -> EXP
Changed lines of the file:
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@@
 		(tags "Through hole pin header THT 2x05 2.54mm double row")
 		(property "Reference" "J3"
-			(at 3.5 -2.9 0)
+			(at 1.13 -2.53 0)
 			(layer "F.SilkS")
 			(effects
@@
 			)
 		)
-		(property "Value" "Conn_02x05_Odd_Even"
-			(at 1.27 12.49 0)
-			(layer "F.Fab")
-			(hide yes)
+		(property "Value" "EXP"
+			(at 1.33 12.64 0)
+			(layer "F.SilkS")
 			(effects
 				(font

Commit message: Remove oscillator from CPU cards
Parts:
- removed X1: OCXO-14, Oscillator:Oscillator_DIP-14
Routing:
- net PHI2: track 98.7 -> 49.0 mm, vias 4 -> 2
- net VCC: track 171.3 -> 165.2 mm, vias 6 -> 5
