File: Hardware/Keypad Expander/Rev 1.0/Keypad Expander.kicad_pcb (KiCad board)
At the start: 2 copper layers, 81.8 x 57.6 mm, 16 parts, among them J1 6502 Card Edge, J2 PORT B, J3 PORT A, U1 65C21, U2 AT28C256, U3 74HC138

Commit message: Update Keypad Expander ROM
Parts:
- U2: value AT28C256 -> AT28C64
Connections:
- U2 pad 1: A14 -> unconnected-(U2-NC-Pad1)
- U2 pad 26: A13 -> unconnected-(U2-NC-Pad26)
Changed lines of the file:
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@@
 	(net 64 "unconnected-(U3-~{Y1}-Pad14)")
 	(net 65 "unconnected-(U3-~{Y0}-Pad15)")
+	(net 66 "unconnected-(U2-NC-Pad1)")
+	(net 67 "unconnected-(U2-NC-Pad26)")
 	(footprint "6502 Logos:6502 Keypad Expander Logo 4mm"
 		(layer "F.Cu")
@@
 			)
 		)
-		(property "Datasheet" ""
+		(property "Datasheet" "~"
 			(at 0 0 0)
 			(unlocked yes)
@@
 			)
 		)
-		(property "Description" ""
+		(property "Description" "Generic connector, double row, 02x06, odd/even pin numbering scheme (row 1 odd numbers, row 2 even numbers), script generated (kicad-library-utils/schlib/autogen/connector/)"
 			(at 0 0 0)
 			(unlocked yes)
@@
 			)
 		)
-		(property "Datasheet" ""
+		(property "Datasheet" "~"
 			(at 0 0 0)
 			(layer "F.Fab")
@@
 			)
 		)
+		(property "LCSC" "C49678"
+			(at 0 0 0)
+			(unlocked yes)
+			(layer "F.Fab")
+			(hide yes)
+			(effects
+				(font
+					(size 1 1)
+					(thickness 0.15)
+				)
+			)
+		)
 		(property ki_fp_filters "C_*")
 		(sheetname "/")
@@
 			)
 		)
-		(property "Value" "AT28C256"
+		(property "Value" "AT28C64"
 			(at 7.62 35.8 90)
 			(layer "F.SilkS")
@@
 		(sheetname "/")
 		(sheetfile "Keypad Expander.kicad_sch")
-		(attr through_hole exclude_from_bom)
+		(attr through_hole)
 		(fp_line
 			(start 13.68 -1.33)
@@
 			(remove_unused_layers no)
 			(roundrect_rratio 0.15625)
-			(net 25 "A14")
-			(pinfunction "A14")
-			(pintype "bidirectional")
+			(net 66 "unconnected-(U2-NC-Pad1)")
+			(pinfunction "NC")
+			(pintype "no_connect")
 		)
 		(pad "2" thru_hole oval
@@
 			(layers "*.Cu" "*.Mask")
 			(remove_unused_layers no)
-			(net 10 "A13")
-			(pinfunction "A13")
-			(pintype "bidirectional")
+			(net 67 "unconnected-(U2-NC-Pad26)")
+			(pinfunction "NC")
+			(pintype "no_connect")
 		)
 		(pad "27" thru_hole oval
@@
 			)
 		)
-		(property "Datasheet" ""
+		(property "Datasheet" "~"
 			(at 0 0 0)
 			(unlocked yes)
@@
 			)
 		)
-		(property "Description" ""
+		(property "Description" "Generic connector, double row, 02x06, odd/even pin numbering scheme (row 1 odd numbers, row 2 even numbers), script generated (kicad-library-utils/schlib/autogen/connector/)"
 			(at 0 0 0)
 			(unlocked yes)

Commit message: Add RWB qualification to Keypad Expander
Parts:
- added C4: 100nF, Capacitor_THT:C_Disc_D5.0mm_W2.5mm_P5.00mm, F.Cu at (90.1, 105.9)
- added U4: 74HC138, Package_DIP:DIP-16_W7.62mm_Socket_LongPads, F.Cu at (78.8, 106.0)
Connections:
- U3 pad 7: REB -> Net-(U3-~{Y7})
