File: Hardware/ROM Cart/Rev 1.0b/ROM Cart.kicad_pcb (KiCad board)
At the start: 2 copper layers, 81.8 x 57.6 mm, 12 parts, among them J1 6502 Card Edge, U1 AT28C256, U2 74HC138

Commit message: Re-version ROM carts
Parts:
- U1: value AT28C256 -> AT27C256
Connections:
- net RB renamed REB
- U1 pad 1: A14 -> unconnected-(U1-VPP-Pad1)
- U1 pad 27: VCC -> A14
Routing:
- net A14: track 34.6 -> 45.2 mm, vias 3 -> 2
Other:
- board text added: "© 2025 A.C. Wright Design | acwrightdesign.com | Rev 1.0b"
- board text removed: "© 2025 A.C. Wright Design | acwrightdesign.com | Rev 0"
Changed lines of the file:
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@@
 	(title_block
 		(title "6502 ROM Cart")
-		(date "2025-09-17")
-		(rev "0.0")
+		(date "2026-03-22")
+		(rev "1.0b")
 		(company "A.C. Wright Design")
 	)
@@
 	)
 	(net 0 "")
-	(net 1 "RB")
+	(net 1 "unconnected-(U1-VPP-Pad1)")
 	(net 2 "A3")
 	(net 3 "A0")
@@
 	(net 43 "unconnected-(J1-PadIRQB)")
 	(net 44 "unconnected-(J1-PadEXP3)")
+	(net 45 "REB")
 	(footprint "6502 Logos:6502 ROM Cart Logo 5mm"
 		(layer "F.Cu")
@@
 			(layers "*.Cu" "*.Mask")
 			(remove_unused_layers no)
-			(net 1 "RB")
+			(net 45 "REB")
 			(pinfunction "~{Y7}")
 			(pintype "output")
@@
 			)
 		)
-		(property "Value" "AT28C256"
+		(property "Value" "AT27C256"
 			(at 7.62 35.8 90)
 			(layer "F.SilkS")
@@
 		(sheetname "/")
 		(sheetfile "ROM Cart.kicad_sch")
-		(attr through_hole exclude_from_bom)
+		(attr through_hole)
 		(fp_line
 			(start 13.68 -1.33)
@@
 			(remove_unused_layers no)
 			(roundrect_rratio 0.15625)
-			(net 25 "A14")
-			(pinfunction "A14")
-			(pintype "bidirectional")
+			(net 1 "unconnected-(U1-VPP-Pad1)")
+			(pinfunction "VPP")
+			(pintype "power_in+no_connect")
 		)
 		(pad "2" thru_hole oval
@@
 			(layers "*.Cu" "*.Mask")
 			(remove_unused_layers no)
-			(net 1 "RB")
+			(net 45 "REB")
 			(pinfunction "~{CE}")
 			(pintype "bidirectional")
@@
 			(layers "*.Cu" "*.Mask")
 			(remove_unused_layers no)
-			(net 1 "RB")
+			(net 45 "REB")
 			(pinfunction "~{OE}")
 			(pintype "bidirectional")
@@
 			(layers "*.Cu" "*.Mask")
 			(remove_unused_layers no)
-			(net 19 "VCC")
-			(pinfunction "~{WE}")
+			(net 25 "A14")
+			(pinfunction "A14")
 			(pintype "bidirectional")
 		)
@@
 		(layer "Edge.Cuts")
 	)
-	(gr_text "© 2025 A.C. Wright Design | acwrightdesign.com | Rev 0"
-		(at 178.6 100.2 90)
+	(gr_text "© 2025 A.C. Wright Design | acwrightdesign.com | Rev 1.0b"
+		(at 178.6111 101.3036 90)
 		(layer "F.SilkS")
 		(effects
@@
 	)
 	(segment
-		(start 123.69 97.31)
-		(end 123.7 97.3)
-		(width 0.25)
-		(layer "F.Cu")
-		(net 1)
-	)
-	(segment
-		(start 116.94 96.33)
-		(end 120.58 96.33)
-		(width 0.25)
-		(layer "F.Cu")
-		(net 1)
-	)
-	(segment
-		(start 121.56 97.31)
-		(end 123.69 97.31)
-		(width 0.25)
-		(layer "F.Cu")
-		(net 1)
-	)
-	(segment
-		(start 137.64 97.26)
-		(end 137.64 93.76)
-		(width 0.25)
-		(layer "F.Cu")
-		(net 1)
-	)
-	(segment
-		(start 120.58 96.33)
-		(end 121.56 97.31)
-		(width 0.25)
-		(layer "F.Cu")
-		(net 1)
-	)
-	(segment
-		(start 137.6 97.3)
-		(end 137.64 97.26)
-		(width 0.25)
-		(layer "F.Cu")
-		(net 1)
-	)
-	(via
-		(at 137.6 97.3)
-		(size 0.8)
-		(drill 0.4)
-		(layers "F.Cu" "B.Cu")
-		(net 1)
-	)
-	(via
-		(at 123.7 97.3)
-		(size 0.8)
-		(drill 0.4)
-		(layers "F.Cu" "B.Cu")
-		(net 1)
-	)
-	(segment
-		(start 142 91.2)
-		(end 142.72 91.92)
-		(width 0.25)
-		(layer "B.Cu")
-		(net 1)
-	)
-	(segment
-		(start 137.64 93.76)
-		(end 137.64 92.06)
-		(width 0.25)
-		(layer "B.Cu")
-		(net 1)
-	)
-	(segment
-		(start 137.64 92.06)
-		(end 138.5 91.2)
-		(width 0.25)
-		(layer "B.Cu")
-		(net 1)
-	)
-	(segment
-		(start 123.7 97.3)
-		(end 137.6 97.3)
-		(width 0.25)
-		(layer "B.Cu")
-		(net 1)
-	)
-	(segment
-		(start 142.72 91.92)
-		(end 142.72 93.76)
-		(width 0.25)
-		(layer "B.Cu")
-		(net 1)
-	)
-	(segment
-		(start 138.5 91.2)
-		(end 142 91.2)
+		(start 122.37 109.03)
+		(end 122.4 109)
 		(width 0.25)
 		(layer "B.Cu")
@@
 	)
 	(segment
-		(start 163.56 123.34)
-		(end 163.56 130.03)
+		(start 122.4411 96.0936)
+		(end 122.4411 93.8011)
 		(width 0.25)
 		(layer "F.Cu")
@@
 	)
 	(segment
-		(start 124.94 93.76)
-		(end 124.94 96.06)
+		(start 163.56 123.34)
+		(end 163.56 130.03)
 		(width 0.25)
 		(layer "F.Cu")
@@
 	)
 	(segment
-		(start 124.94 96.06)
-		(end 124.9 96.1)
+		(start 122.4411 93.8011)
+		(end 122.4 93.76)
 		(width 0.25)
 		(layer "F.Cu")
@@
 	)
 	(via
-		(at 124.9 96.1)
+		(at 163.6 96)
 		(size 0.8)
 		(drill 0.4)
@@
 	)
 	(via
-		(at 163.6 96)
+		(at 122.4411 96.0936)
 		(size 0.8)
 		(drill 0.4)
@@
 	)
 	(segment
+		(start 124.9 96.1)
+		(end 122.4475 96.1)
+		(width 0.25)
+		(layer "B.Cu")
+		(net 19)
+	)
+	(segment
 		(start 163.5 96.1)
 		(end 163.6 96)
@@
 	)
 	(segment
+		(start 122.4475 96.1)
+		(end 122.4411 96.0936)
+		(width 0.25)
+		(layer "B.Cu")
+		(net 19)
+	)
+	(segment
 		(start 115.3 130.03)
 		(end 115.3 123.27)
@@
 	)
 	(segment
-		(start 122.4 93.76)
-		(end 124.94 93.76)
-		(width 0.25)
-		(layer "B.Cu")
-		(net 19)
-	)
-	(segment
 		(start 115.29 121.19)
 		(end 110.9 116.8)
@@
 	)
 	(segment
-		(start 122.4 112.05)
-		(end 122.4 111.3)
+		(start 123.6711 105.9836)
+		(end 123.6711 106.8636)
 		(width 0.25)
 		(layer "F.Cu")
@@
 	)
 	(segment
-		(start 129.1 111.3)
-		(end 129.15 111.35)
+		(start 125.47 115.16)
+		(end 125.49 115.14)
 		(width 0.25)
 		(layer "F.Cu")
@@
 	)
 	(segment
-		(start 125.47 115.16)
+		(start 123.6711 113.3211)
 		(end 125.49 115.14)
 		(width 0.25)
@@
 	)
 	(segment
-		(start 122.4 109)
-		(end 122.4 111.3)
+		(start 124.94 93.76)
+		(end 124.94 104.7147)
 		(width 0.25)
 		(layer "F.Cu")
@@
 	)
 	(segment
-		(start 125.49 115.14)
-		(end 122.4 112.05)
+		(start 124.94 104.7147)
+		(end 123.6711 105.9836)
 		(width 0.25)
 		(layer "F.Cu")
@@
 	)
 	(segment
-		(start 125.47 125.12)
-		(end 125.47 115.16)
+		(start 123.6711 106.8636)
+		(end 123.6711 113.3211)
 		(width 0.25)
 		(layer "F.Cu")
 		(net 25)
 	)
-	(via
-		(at 129.1 111.3)
-		(size 0.8)
-		(drill 0.4)
-		(layers "F.Cu" "B.Cu")
+	(segment
+		(start 125.47 125.12)
+		(end 125.47 115.16)
+		(width 0.25)
+		(layer "F.Cu")
 		(net 25)
 	)
@@
 	)
 	(via
-		(at 122.4 111.3)
+		(at 123.6711 106.8636)
 		(size 0.8)
 		(drill 0.4)
@@
 	)
 	(segment
-		(start 122.4 111.3)
-		(end 129.1 111.3)
+		(start 118.6647 109.03)
+		(end 120.8311 106.8636)
 		(width 0.25)
 		(layer "B.Cu")
@@
 	)
 	(segment
-		(start 116.94 109.03)
-		(end 122.37 109.03)
+		(start 120.8311 106.8636)
+		(end 123.6711 106.8636)
 		(width 0.25)
 		(layer "B.Cu")
@@
 	)
 	(segment
-		(start 122.37 109.03)
-		(end 122.4 109)
+		(start 116.94 109.03)
+		(end 118.6647 109.03)
 		(width 0.25)
 		(layer "B.Cu")
@@
 		(net 36)
 	)
+	(segment
+		(start 123.69 97.31)
+		(end 123.7 97.3)
+		(width 0.25)
+		(layer "F.Cu")
+		(net 45)
+	)
+	(segment
+		(start 116.94 96.33)
+		(end 120.58 96.33)
+		(width 0.25)
+		(layer "F.Cu")
+		(net 45)
+	)
+	(segment
+		(start 121.56 97.31)
+		(end 123.69 97.31)
+		(width 0.25)
+		(layer "F.Cu")
+		(net 45)
+	)
+	(segment
+		(start 137.64 97.26)
+		(end 137.64 93.76)
+		(width 0.25)
+		(layer "F.Cu")
+		(net 45)
+	)
+	(segment
+		(start 120.58 96.33)
+		(end 121.56 97.31)
+		(width 0.25)
+		(layer "F.Cu")
+		(net 45)
+	)
+	(segment
+		(start 137.6 97.3)
+		(end 137.64 97.26)
+		(width 0.25)
+		(layer "F.Cu")
+		(net 45)
+	)
+	(via
+		(at 137.6 97.3)
+		(size 0.8)
+		(drill 0.4)
+		(layers "F.Cu" "B.Cu")
+		(net 45)
+	)
+	(via
+		(at 123.7 97.3)
+		(size 0.8)
+		(drill 0.4)
+		(layers "F.Cu" "B.Cu")
+		(net 45)
+	)
+	(segment
+		(start 142 91.2)
+		(end 142.72 91.92)
+		(width 0.25)
+		(layer "B.Cu")
+		(net 45)
+	)
+	(segment
+		(start 137.64 93.76)
+		(end 137.64 92.06)
+		(width 0.25)
+		(layer "B.Cu")
+		(net 45)
+	)
+	(segment
+		(start 137.64 92.06)
+		(end 138.5 91.2)
+		(width 0.25)
+		(layer "B.Cu")
+		(net 45)
+	)
+	(segment
+		(start 123.7 97.3)
+		(end 137.6 97.3)
+		(width 0.25)
+		(layer "B.Cu")
+		(net 45)
+	)
+	(segment
+		(start 142.72 91.92)
+		(end 142.72 93.76)
+		(width 0.25)
+		(layer "B.Cu")
+		(net 45)
+	)
+	(segment
+		(start 138.5 91.2)
+		(end 142 91.2)
+		(width 0.25)
+		(layer "B.Cu")
+		(net 45)
+	)
 	(zone
